File: Hardware/LED_Module/Microcontroller.kicad_sch (KiCad schematic)
At the start: 30 parts, among them J4001 USB_C_Receptacle_USB2.0_16P, J4002 TagConnect_SWD, SW4001 SW_Push, SW4002 SW_Push, U4001 W25Q64JVXGIQ, U4002 RP2040, Y4001 12M

Commit message: User interface fix
Parts:
- renumbered C4001 to C401, C4002 to C402, C4003 to C403, C4004 to C404, C4005 to C405, C4006 to C406, C4007 to C407, C4008 to C408, C4009 to C409, C4010 to C410, C4011 to C411, C4012 to C412, C4013 to C413, C4014 to C414, C4015 to C415, D4001 to D401, J4001 to J401, J4002 to J402, R4001 to R401, R4002 to R402, R4003 to R403, R4004 to R404, R4005 to R405, R4006 to R406, R4007 to R407, SW4001 to SW401, SW4002 to SW402, U4001 to U401, U4002 to U402, Y4001 to Y401

Commit message: Changes and fixes
Parts:
- Y401: footprint Crystal:Crystal_SMD_Abracon_ABM3B-4Pin_5.0x3.2mm -> Crystal:Crystal_SMD_2520-4Pin_2.5x2.0mm; mouser 815-ABM3B1210B1UT -> 520-120-10-36Q-AEST
Changed lines of the file:
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@@
-	)
-	(symbol
-		(lib_id "Device:Crystal_GND24")
-		(at 44.45 148.59 90)
-		(unit 1)
-		(exclude_from_sim no)
-		(in_bom yes)
-		(on_board yes)
-		(dnp no)
-		(property "Reference" "Y401"
-			(at 44.45 138.43 90)
-			(effects
-				(font
-					(size 1.27 1.27)
-				)
-			)
-		)
-		(property "Value" "12M"
-			(at 44.45 140.97 90)
-			(effects
-				(font
-					(size 1.27 1.27)
-				)
-			)
-		)
-		(property "Footprint" "Crystal:Crystal_SMD_Abracon_ABM3B-4Pin_5.0x3.2mm"
-			(at 44.45 148.59 0)
-			(effects
-				(font
-					(size 1.27 1.27)
-				)
-				(hide yes)
-			)
-		)
-		(property "Datasheet" "https://eu.mouser.com/datasheet/2/3/abm3b-1774998.pdf"
-			(at 44.45 148.59 0)
-			(effects
-				(font
-					(size 1.27 1.27)
-				)
-				(hide yes)
-			)
-		)
-		(property "Description" ""
-			(at 44.45 148.59 0)
-			(effects
-				(font
-					(size 1.27 1.27)
-				)
-				(hide yes)
-			)
-		)
-		(property "mouser" "815-ABM3B1210B1UT"
-			(at 44.45 148.59 0)
-			(effects
-				(font
-					(size 1.27 1.27)
-				)
-				(hide yes)
-			)
-		)
-		(property "ETA" ""
-			(at 44.45 148.59 0)
-			(effects
-				(font
-					(size 1.27 1.27)
-				)
-				(hide yes)
-			)
-		)
-		(property "REASON" "ABM3B-12.000MHZ-10-B-1-U-T  is not sold at RS or elfa"
-			(at 44.45 148.59 0)
-			(effects
-				(font
-					(size 1.27 1.27)
-				)
-				(hide yes)
-			)
-		)
-		(property "RS-COMPONENTS" ""
-			(at 44.45 148.59 0)
-			(effects
-				(font
-					(size 1.27 1.27)
-				)
-				(hide yes)
-			)
-		)
-		(property "Footprint checked" "YES"
-			(at 44.45 148.59 0)
-			(effects
-				(font
-					(size 1.27 1.27)
-				)
-				(hide yes)
-			)
-		)
-		(pin "1"
-		)
-		(pin "2"
-		)
-		(pin "4"
-		)
-		(pin "3"
-		)
-		(instances
-			(project "LED_Module"
-				(path "/16808901-367a-4ed1-b5c3-f1221533388f/491ba666-eea9-4d2d-9b48-12ddc2954e77"
-					(reference "Y401")
-					(unit 1)
-				)
-			)
-			(project "Ficklampa"
-				(path "/ddeb2498-781c-4bfa-9a76-a6e5959b49e0"
-					(reference "Y101")
-					(unit 1)
-				)
-			)
-			(project "JBCock"
-				(path "/e866f8fb-0ce5-4a7b-98ed-8451088f137a"
-					(reference "Y101")
-					(unit 1)
-				)
-			)
-		)
 	)
 	(symbol
@@
 					(unit 1)
 				)
+			)
+		)
+	)
+	(symbol
+		(lib_id "Device:Crystal_GND24")
+		(at 44.45 148.59 90)
+		(unit 1)
+		(exclude_from_sim no)
+		(in_bom yes)
+		(on_board yes)
+		(dnp no)
+		(property "Reference" "Y401"
+			(at 44.45 138.43 90)
+			(effects
+				(font
+					(size 1.27 1.27)
+				)
+			)
+		)
+		(property "Value" "12M"
+			(at 44.45 140.97 90)
+			(effects
+				(font
+					(size 1.27 1.27)
+				)
+			)
+		)
+		(property "Footprint" "Crystal:Crystal_SMD_2520-4Pin_2.5x2.0mm"
+			(at 44.45 148.59 0)
+			(effects
+				(font
+					(size 1.27 1.27)
+				)
+				(hide yes)
+			)
+		)
+		(property "Datasheet" "https://www.mouser.se/datasheet/2/122/ECX_2236Q-938171.pdf"
+			(at 44.45 148.59 0)
+			(effects
+				(font
+					(size 1.27 1.27)
+				)
+				(hide yes)
+			)
+		)
+		(property "Description" ""
+			(at 44.45 148.59 0)
+			(effects
+				(font
+					(size 1.27 1.27)
+				)
+				(hide yes)
+			)
+		)
+		(property "mouser" "520-120-10-36Q-AEST"
+			(at 44.45 148.59 0)
+			(effects
+				(font
+					(size 1.27 1.27)
+				)
+				(hide yes)
+			)
+		)
+		(property "ETA" ""
+			(at 44.45 148.59 0)
+			(effects
+				(font
+					(size 1.27 1.27)
+				)
+				(hide yes)
+			)
+		)
+		(property "REASON" "ABM3B-12.000MHZ-10-B-1-U-T  is not sold at RS or elfa"
+			(at 44.45 148.59 0)
+			(effects
+				(font
+					(size 1.27 1.27)
+				)
+				(hide yes)
+			)
+		)
+		(property "RS-COMPONENTS" ""
+			(at 44.45 148.59 0)
+			(effects
+				(font
+					(size 1.27 1.27)
+				)
+				(hide yes)
+			)
+		)
+		(property "Footprint checked" "YES"
+			(at 44.45 148.59 0)
+			(effects
+				(font
+					(size 1.27 1.27)
+				)
+				(hide yes)
+			)
+		)
+		(pin "1"
+		)
+		(pin "2"
+		)
+		(pin "4"
+		)
+		(pin "3"
+		)
+		(instances
+			(project "LED_Module"
+				(path "/16808901-367a-4ed1-b5c3-f1221533388f/491ba666-eea9-4d2d-9b48-12ddc2954e77"
+					(reference "Y401")
+					(unit 1)
+				)

Commit message: final fixes (hopefully) (GONE WRONG?!) (real)
Other:
- title: (none) -> RP2040 Microcontroller and support components
Changed lines of the file:
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@@
 	(paper "A4")
 	(title_block
+		(title "RP2040 Microcontroller and support components")
+		(date "2024-03-26")
+		(rev "B01")
 		(company "Chalmers EENX16-VT24-27")
 	)
