File: Hardware/LED_Module/CAN_bus.kicad_sch (KiCad schematic)
At the start: 13 parts, among them J2 RJ10, J3 RJ10, U6 MCP2515-xST, U7 MCP2551-I-SN, Y2 8M

Commit message: La in allt
Myyycket saker
Parts:
- added C2001, C2002: 10u, Capacitor_SMD:C_1206_3216Metric, symbol Device:C
- added C2003, C2004: 100n, Capacitor_SMD:C_0402_1005Metric, symbol Device:C
- added F2001: 4A, Fuse:Fuse_0603_1608Metric, symbol Device:Fuse
- added TP2001: TPVin, TestPoint:TestPoint_Pad_D2.0mm, symbol Connector:TestPoint
- C2005: renamed from C14; value C -> 10p; footprint (none) -> Capacitor_SMD:C_0402_1005Metric; Footprint checked (none) -> YES; mouser (none) -> 81-GRT1555C2A100JA2J
- C2006: renamed from C20; value C -> 10p; footprint (none) -> Capacitor_SMD:C_0402_1005Metric; Footprint checked (none) -> YES; mouser (none) -> 81-GRT1555C2A100JA2J
- J2001: renamed from J2; value RJ10 -> RJ9; Footprint checked (none) -> YES; mouser (none) -> 649-61835-0441LF
- J2002: renamed from J3; value RJ10 -> RJ9; Footprint checked (none) -> YES; mouser (none) -> 649-61835-0441LF
- JP2001: renamed from JP2; footprint (none) -> Connector_PinHeader_2.54mm:PinHeader_1x02_P2.54mm_Vertical; ETA (none) -> ETA; Footprint checked (none) -> YES
- R2001: renamed from R15; footprint (none) -> Resistor_SMD:R_0402_1005Metric; Footprint checked (none) -> YES; mouser (none) -> 71-CRCW0402J-120-E3
- R2002: renamed from R12; value 5k -> 5k1; footprint (none) -> Resistor_SMD:R_0402_1005Metric; Footprint checked (none) -> YES; mouser (none) -> 71-CRCW0402-5.1K-E3
- R2003: renamed from R13; footprint (none) -> Resistor_SMD:R_0402_1005Metric; Footprint checked (none) -> YES; mouser (none) -> 71-CRCW040210K0JNEDC
- R2004: renamed from R14; footprint (none) -> Resistor_SMD:R_0402_1005Metric; Footprint checked (none) -> YES; mouser (none) -> 71-CRCW040210K0JNEDC
- R2005: renamed from R6; footprint (none) -> Resistor_SMD:R_0402_1005Metric; Footprint checked (none) -> YES; mouser (none) -> 71-CRCW040210K0JNEDC
- U2001: renamed from U7; ETA (none) -> ETA; Footprint checked (none) -> YES
- U2002: renamed from U6; ETA (none) -> ETA; Footprint checked (none) -> YES
- Y2001: renamed from Y2; footprint (none) -> Crystal:Crystal_SMD_Abracon_ABM3B-4Pin_5.0x3.2mm; Footprint checked (none) -> YES; REASON (none) -> ABM3B-8.000MHZ-10-1-U-T is not sold at RS or elfa; mouser (none) -> 815-ABM3B8MHZ101UT
Connections:
- net +3V3: now also C2003.1
- net +5V: now also C2004.1
- net GND: now also C2001.2, C2002.2, C2003.2, C2004.2
- net +IN_BATT: no longer names the net of J2001.4, J2002.4
- net +IN_BATT: now also F2001.1
- new net +SYSTEM: C2001.1, C2002.1, F2001.2, TP2001.1
Other:
- company: (none) -> Chalmers EENX16-VT24-27

Commit message: User interface fix
Parts:
- renumbered C2001 to C201, C2002 to C202, C2003 to C203, C2004 to C204, C2005 to C205, C2006 to C206, F2001 to F201, J2001 to J201, J2002 to J202, JP2001 to JP201, R2001 to R201, R2002 to R202, R2003 to R203, R2004 to R204, R2005 to R205, TP2001 to TP201, U2001 to U201, U2002 to U202, Y2001 to Y201

Commit message: LED module go brrrrrrrrrrrrrrrrrr
Parts:
- Y201: symbol Device:Crystal_GND23 -> Device:Crystal_GND24
Connections:
- net GND: now also Y201.4; no longer Y201.3
- net at C205.2, U202.8 (OSC2): now also Y201.3; no longer Y201.4
Changed lines of the file:
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@@
 	)
 	(symbol
-		(lib_id "Device:Crystal_GND23")
+		(lib_id "Device:Crystal_GND24")
 		(at 60.96 105.41 90)
 		(unit 1)
@@
 			)
 		)
-		(property "Datasheet" "https://www.mouser.se/datasheet/2/3/abm3b-1774998.pdf"
+		(property "Datasheet" "~"
 			(at 60.96 105.41 0)
 			(effects
@@
 			)
 		)
-		(property "Description" ""
+		(property "Description" "Four pin crystal, GND on pins 2 and 4"
 			(at 60.96 105.41 0)
 			(effects

Commit message: User interface and Controller done
yes
Parts:
- C201, C202: footprint Capacitor_SMD:C_1206_3216Metric -> Capacitor_SMD:C_0805_2012Metric; mouser 581-1206DD106MAT2A -> 81-GRM21BR61H106KE3L
Changed lines of the file:
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@@
 			)
 		)
-		(property "Footprint" "Capacitor_SMD:C_1206_3216Metric"
+		(property "Footprint" "Capacitor_SMD:C_0805_2012Metric"
 			(at 249.8852 53.34 0)
 			(effects
@@
 			)
 		)
-		(property "Datasheet" "https://www.mouser.se/datasheet/2/40/cx5r_KGM-3223198.pdf"
+		(property "Datasheet" ""
 			(at 248.92 49.53 0)
 			(effects
@@
 			)
 		)
-		(property "mouser" "581-1206DD106MAT2A"
+		(property "mouser" "81-GRM21BR61H106KE3L"
 			(at 248.92 49.53 0)
 			(effects
@@
 			)
 		)
-		(property "Footprint" "Capacitor_SMD:C_1206_3216Metric"
+		(property "Footprint" "Capacitor_SMD:C_0805_2012Metric"
 			(at 239.7252 53.34 0)
 			(effects
@@
 			)
 		)
-		(property "Datasheet" "https://www.mouser.se/datasheet/2/40/cx5r_KGM-3223198.pdf"
+		(property "Datasheet" ""
 			(at 238.76 49.53 0)
 			(effects
@@
 			)
 		)
-		(property "mouser" "581-1206DD106MAT2A"
+		(property "mouser" "81-GRM21BR61H106KE3L"
 			(at 238.76 49.53 0)
 			(effects

Commit message: final fixes (hopefully) (GONE WRONG?!) (real)
Other:
- title: (none) -> CAN Bus controller + interface
Changed lines of the file:
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@@
 	(paper "A4")
 	(title_block
+		(title "CAN Bus controller + interface")
+		(date "2024-03-26")
+		(rev "B01")
 		(company "Chalmers EENX16-VT24-27")
 	)
