File: Hardware/LED_Module/LED_Module.kicad_pcb (KiCad board)
At the start: 2 copper layers, 50 x 70 mm, 38 parts, among them J1 TagConnect_SWD, J2 RJ10, J3 RJ10, J4 USB_C_Receptacle, SW1 SW_Push, U1 W25Q64JVXGIQ, U2 RP2040, U3 LTC7001, U4 LT8653S, U5 CH224K, Y1 Crystal

Commit message: La in allt
Myyycket saker
Parts:
- removed C1, C10, C11, C12, C13, C15, C16, C5, C6, C7, C8, C9: 100n, Capacitor_SMD:C_0402_1005Metric
- removed C14: 2200p, personal:C_feedthrough_0805
- removed C17, C18, C19: 10u, Capacitor_SMD:C_0805_2012Metric
- removed C2, C3: 10p, Capacitor_SMD:C_0402_1005Metric
- removed C4: 1u, Capacitor_SMD:C_0402_1005Metric
- removed J1: TagConnect_SWD, Connector:Tag-Connect_TC2030-IDC-NL_2x03_P1.27mm_Vertical
- removed J2, J3: RJ10, Connector_RJ:RJ9_Evercom_5301-440xxx_Horizontal
- removed J4: USB_C_Receptacle, Connector_USB:USB_C_Receptacle_Amphenol_12401548E4-2A
- removed L1, L2: 2.2u, Inductor_SMD:L_Bourns_SRP7028A_7.3x6.6mm
- removed R1, R5: 1k, Resistor_SMD:R_0402_1005Metric
- removed R2, R3, R6: 27, Resistor_SMD:R_0402_1005Metric
- removed R4: 10k, Resistor_SMD:R_0402_1005Metric
- removed SW1: SW_Push, Button_Switch_SMD:SW_Push_SPST_NO_Alps_SKRK
- removed U1: W25Q64JVXGIQ, Package_SON:WSON-8-1EP_4x4mm_P0.8mm_EP2.2x3mm
- removed U2: RP2040, Package_DFN_QFN:QFN-56-1EP_7x7mm_P0.4mm_EP3.2x3.2mm
- removed U3: LTC7001, Package_SO:MSOP-10-1EP_3x3mm_P0.5mm_EP1.68x1.88mm_ThermalVias
- removed U4: LT8653S, Package_DFN_QFN:QFN-20-1EP_3x4mm_P0.5mm_EP1.65x2.65mm_ThermalVias
- removed U5: CH224K, WCH:ESSOP10
- removed Y1: Crystal, Crystal:Crystal_SMD_Abracon_ABM3B-4Pin_5.0x3.2mm
- added C2001: 10u, Capacitor_SMD:C_1206_3216Metric, F.Cu at (88.0, 46.0)
- added C2002: 10u, Capacitor_SMD:C_1206_3216Metric, F.Cu at (88.0, 43.6)
- added C2003: 100n, Capacitor_SMD:C_0402_1005Metric, F.Cu at (68.9, 21.1)
- added C2004: 100n, Capacitor_SMD:C_0402_1005Metric, F.Cu at (68.9, 23.0)
- added C2005: 10p, Capacitor_SMD:C_0402_1005Metric, F.Cu at (68.9, 25.0)
- added C2006: 10p, Capacitor_SMD:C_0402_1005Metric, F.Cu at (68.9, 27.0)
- added C3001: 100n, Capacitor_SMD:C_0402_1005Metric, F.Cu at (86.2, 55.5)
- added C3002: 10u, Capacitor_SMD:C_1206_3216Metric, F.Cu at (88.8, 51.8)
- added C3003: 22u, Capacitor_SMD:C_0805_2012Metric, F.Cu at (92.2, 55.2)
- added C3004: 22u, Capacitor_SMD:C_0805_2012Metric, F.Cu at (94.2, 55.2)
- added C3005: 100n, Capacitor_SMD:C_0402_1005Metric, F.Cu at (100.5, 55.8)
- added C3006: 10u, Capacitor_SMD:C_1206_3216Metric, F.Cu at (103.0, 52.0)
- added C3007: 22u, Capacitor_SMD:C_0805_2012Metric, F.Cu at (106.5, 55.5)
- added C3008: 22u, Capacitor_SMD:C_0805_2012Metric, F.Cu at (108.5, 55.5)
- added C4001: 100n, Capacitor_SMD:C_0402_1005Metric, F.Cu at (73.8, 78.1)
- added C4002: 100n, Capacitor_SMD:C_0402_1005Metric, F.Cu at (73.8, 80.1)
- added C4003: 100n, Capacitor_SMD:C_0402_1005Metric, F.Cu at (74.0, 82.1)
- added C4004: 100n, Capacitor_SMD:C_0402_1005Metric, F.Cu at (73.8, 84.0)
- added C4005: 100n, Capacitor_SMD:C_0402_1005Metric, F.Cu at (73.8, 86.0)
- added C4006: 100n, Capacitor_SMD:C_0402_1005Metric, F.Cu at (73.8, 88.0)
- added C4007: 100n, Capacitor_SMD:C_0402_1005Metric, F.Cu at (76.7, 78.1)
- added C4008: 100n, Capacitor_SMD:C_0402_1005Metric, F.Cu at (76.7, 80.1)
- added C4009: 100n, Capacitor_SMD:C_0402_1005Metric, F.Cu at (76.7, 82.1)
- added C4010: 1u, Capacitor_SMD:C_0402_1005Metric, F.Cu at (76.7, 84.0)
- added C4011: 100n, Capacitor_SMD:C_0402_1005Metric, F.Cu at (76.7, 86.0)
- added C4012: 100n, Capacitor_SMD:C_0402_1005Metric, F.Cu at (76.7, 88.0)
- added C4013: 100n, Capacitor_SMD:C_0402_1005Metric, F.Cu at (79.5, 78.1)
- added C4014: 10p, Capacitor_SMD:C_0402_1005Metric, F.Cu at (79.5, 80.1)
- added C4015: 10p, Capacitor_SMD:C_0402_1005Metric, F.Cu at (79.5, 82.1)
- added C5001: 10u, Capacitor_SMD:C_1206_3216Metric, F.Cu at (234.8, 47.4)
- added C5002: 100n, Capacitor_SMD:C_0402_1005Metric, F.Cu at (239.0, 64.1)
- added C5003: 10u, Capacitor_SMD:C_1206_3216Metric, F.Cu at (234.8, 50.8)
- added C5004: 100n, Capacitor_SMD:C_0402_1005Metric, F.Cu at (239.0, 66.1)
- added C5005: 100n, Capacitor_SMD:C_0402_1005Metric, F.Cu at (239.0, 68.0)
- added C5006: 100n, Capacitor_SMD:C_0402_1005Metric, F.Cu at (239.0, 70.0)
- added C5007: 10u, Capacitor_SMD:C_1206_3216Metric, F.Cu at (234.8, 54.1)
- added C5008: 10u, Capacitor_SMD:C_1206_3216Metric, F.Cu at (234.8, 57.5)
- added C5009: 10u, Capacitor_SMD:C_1206_3216Metric, F.Cu at (234.8, 60.8)
- added C5010: 100n, Capacitor_SMD:C_0402_1005Metric, F.Cu at (239.0, 72.0)
- added C5011: 100n, Capacitor_SMD:C_0402_1005Metric, F.Cu at (239.0, 74.0)
- added C5012: 10u, Capacitor_SMD:C_1206_3216Metric, F.Cu at (234.8, 64.2)
- added C5013: 100n, Capacitor_SMD:C_0402_1005Metric, F.Cu at (239.0, 75.9)
- added C6001: 100n, Capacitor_SMD:C_0402_1005Metric, F.Cu at (184.8, 82.0)
- added C6002: 100n, Capacitor_SMD:C_0402_1005Metric, F.Cu at (179.5, 84.0)
- added D4001: D_Schottky, Diode_SMD:Nexperia_DSN1608-2_1.6x0.8mm, F.Cu at (91.9, 88.3)
- added D5001: LED-red, footprints:KR DMLQ32. 23, F.Cu at (272.5, 69.7)
- added D5002: LED-main, footprints:LUXEON 7070, F.Cu at (255.8, 50.0)
- added D5003: LED-red, footprints:KR DMLQ32. 23, F.Cu at (276.3, 69.7)
- added D5004: LED-red, footprints:KR DMLQ32. 23, F.Cu at (280.1, 69.7)
- added D5005: LED-red, footprints:KR DMLQ32. 23, F.Cu at (283.9, 69.7)
- added D5006: LED-amber, LED_SMD:LED_PLCC_2835, F.Cu at (240.4, 47.9)
- added D5007: LED-amber, LED_SMD:LED_PLCC_2835, F.Cu at (240.4, 52.2)
- added D5008: LED-amber, LED_SMD:LED_PLCC_2835, F.Cu at (240.4, 56.6)
- added D5009: LED-amber, LED_SMD:LED_PLCC_2835, F.Cu at (240.4, 61.0)
- added D6001: R, LED_SMD:LED_0603_1608Metric, F.Cu at (57.2, 94.9)
- added D6002: G, LED_SMD:LED_0603_1608Metric, F.Cu at (57.2, 97.5)
- added D6003: B, LED_SMD:LED_0603_1608Metric, F.Cu at (57.2, 100.0)
- added F2001: 4A, Fuse:Fuse_0603_1608Metric, F.Cu at (91.2, 44.5)
- added J2001: RJ9, Connector_RJ:RJ9_Evercom_5301-440xxx_Horizontal, F.Cu at (115.8, 42.2)
- added J2002: RJ9, Connector_RJ:RJ9_Evercom_5301-440xxx_Horizontal, F.Cu at (100.1, 42.2)
- added J4001: USB_C_Receptacle_USB2.0_16P, Connector_USB:USB_C_Receptacle_GCT_USB4105-xx-A_16P_TopMnt_Horizontal, F.Cu at (129.3, 38.0)
- added J4002: TagConnect_SWD, Connector:Tag-Connect_TC2030-IDC-NL_2x03_P1.27mm_Vertical, F.Cu at (76.4, 100.4)
- added JP2001: Jumper_termination, Connector_PinHeader_2.54mm:PinHeader_1x02_P2.54mm_Vertical, F.Cu at (88.0, 40.3)
- added L3001: 4u7, Inductor_SMD:L_1210_3225Metric, F.Cu at (90.0, 63.8)
- added L3002: 4u7, Inductor_SMD:L_1210_3225Metric, F.Cu at (104.2, 64.0)
- added L5001: 20u, Inductor_SMD:L_Changjiang_FNR5045S, F.Cu at (246.5, 49.0)
- added L5002: 15u, Inductor_SMD:L_TDK_VLS6045EX_VLS6045AF, F.Cu at (259.1, 62.8)
- added L5003: 5.6u, Inductor_SMD:L_Changjiang_FNR5045S, F.Cu at (246.5, 55.7)
- added R2001: 120, Resistor_SMD:R_0402_1005Metric, F.Cu at (90.8, 38.0)
- added R2002: 5k1, Resistor_SMD:R_0402_1005Metric, F.Cu at (68.9, 13.1)
- added R2003: 10k, Resistor_SMD:R_0402_1005Metric, F.Cu at (68.9, 15.1)
- added R2004: 10k, Resistor_SMD:R_0402_1005Metric, F.Cu at (68.9, 17.1)
- added R2005: 10k, Resistor_SMD:R_0402_1005Metric, F.Cu at (68.9, 19.1)
- added R4001: 5k1, Resistor_SMD:R_0402_1005Metric, F.Cu at (67.2, 78.1)
- added R4002: 5k1, Resistor_SMD:R_0402_1005Metric, F.Cu at (67.2, 80.1)
- added R4003: 10k, Resistor_SMD:R_0402_1005Metric, F.Cu at (67.2, 82.1)
- added R4004: 1k, Resistor_SMD:R_0402_1005Metric, F.Cu at (67.2, 84.1)
- added R4005: 27, Resistor_SMD:R_0402_1005Metric, F.Cu at (67.2, 86.1)
- added R4006: 27, Resistor_SMD:R_0402_1005Metric, F.Cu at (67.2, 88.1)
- added R4007: 1k, Resistor_SMD:R_0402_1005Metric, F.Cu at (67.2, 90.1)
- added R5001: 100m, Resistor_SMD:R_0805_2012Metric, F.Cu at (255.2, 73.1)
- added R5002: 200m, Resistor_SMD:R_1206_3216Metric, F.Cu at (246.0, 68.8)
- added R5003: 200m, Resistor_SMD:R_1206_3216Metric, F.Cu at (246.0, 72.0)
- added R6001: 5k1, Resistor_SMD:R_0402_1005Metric, F.Cu at (176.8, 82.0)
- added R6002: 5k1, Resistor_SMD:R_0402_1005Metric, F.Cu at (177.8, 82.0)
- added R6003: 120, Resistor_SMD:R_0402_1005Metric, F.Cu at (54.8, 95.0)
- added R6004: 120, Resistor_SMD:R_0402_1005Metric, F.Cu at (54.8, 97.5)
- added R6005: 120, Resistor_SMD:R_0402_1005Metric, F.Cu at (54.8, 100.0)
- added SW4001: SW_Push, Button_Switch_SMD:SW_Push_SPST_NO_Alps_SKRK, F.Cu at (129.8, 64.2)
- added SW4002: SW_Push, Button_Switch_SMD:SW_Push_SPST_NO_Alps_SKRK, F.Cu at (75.6, 95.6)
- added TP2001: TPVin, TestPoint:TestPoint_Pad_D2.0mm, F.Cu at (89.5, 48.8)
- added TP3001: TP3V3, TestPoint:TestPoint_Pad_D2.0mm, F.Cu at (96.8, 55.8)
- added TP3002: TP5V, TestPoint:TestPoint_Pad_D2.0mm, F.Cu at (111.2, 56.0)
- added TP5001: TPLED2+, TestPoint:TestPoint_Pad_D2.0mm, F.Cu at (245.2, 61.0)
- added TP5002: TPLED1+, TestPoint:TestPoint_Pad_D2.0mm, F.Cu at (245.2, 65.1)
- added TP5003: TPLED1-, TestPoint:TestPoint_Pad_D2.0mm, F.Cu at (249.2, 61.0)
- added TP5004: TPLED2-, TestPoint:TestPoint_Pad_D2.0mm, F.Cu at (249.2, 65.1)
- added TP5005: TPLED3+, TestPoint:TestPoint_Pad_D2.0mm, F.Cu at (253.3, 61.0)
- added TP5006: TPLED3-, TestPoint:TestPoint_Pad_D2.0mm, F.Cu at (253.3, 65.1)
- added U2001: MCP2551-I-SN, Package_SO:SOIC-8_3.9x4.9mm_P1.27mm, F.Cu at (54.5, 33.5)
- added U2002: MCP2515-xST, Package_SO:TSSOP-20_4.4x6.5mm_P0.65mm, F.Cu at (45.9, 34.2)
- added U3001: AP63203WU, Package_TO_SOT_SMD:TSOT-23-6, F.Cu at (88.9, 55.0)
- added U3002: AP63205WU, Package_TO_SOT_SMD:TSOT-23-6, F.Cu at (103.2, 55.3)
- added U4001: W25Q64JVXGIQ, Package_SON:WSON-8-1EP_4x4mm_P0.8mm_EP2.2x3mm, F.Cu at (119.2, 51.0)
- added U4002: RP2040, Package_DFN_QFN:QFN-56-1EP_7x7mm_P0.4mm_EP3.2x3.2mm, F.Cu at (124.2, 58.0)
- added U5001: TPS92200, footprints:VQFN-HR-6pin-TexasInstruments, F.Cu at (251.7, 47.3)
- added U5002: TPS92200, footprints:VQFN-HR-6pin-TexasInstruments, F.Cu at (251.7, 50.5)
- added U5003: TPS92200, footprints:VQFN-HR-6pin-TexasInstruments, F.Cu at (251.7, 53.7)
- added U5004: TMP236, Package_TO_SOT_SMD:SOT-353_SC-70-5, F.Cu at (250.9, 73.6)
- added U6001: MC3479, footprints:MC3479, F.Cu at (182.8, 81.8)
- added U6002: LTR-303ALS-01, OptoDevice:Lite-On_LTR-303ALS-01, F.Cu at (179.5, 82.0)
- added Y2001: 8M, Crystal:Crystal_SMD_Abracon_ABM3B-4Pin_5.0x3.2mm, F.Cu at (54.0, 39.4)
- added Y4001: Crystal, Crystal:Crystal_SMD_Abracon_ABM3B-4Pin_5.0x3.2mm, F.Cu at (121.5, 67.0)
Routing:
- net /Microcontroller/FLASH_~{CS}: track 0.00 -> 10.5 mm
- net /Microcontroller/FLASH_IO1: track 0.00 -> 9.55 mm
- net /Microcontroller/FLASH_IO2: track 0.00 -> 8.94 mm
- net /SCL: track 0.00 -> 6.17 mm
- net /Microcontroller/FLASH_IO3: track 0.00 -> 5.54 mm
- net /SDA: track 0.00 -> 5.03 mm
- net /Microcontroller/FLASH_CLK: track 0.00 -> 4.60 mm
- net /Microcontroller/FLASH_IO0: track 0.00 -> 3.67 mm
- net +3V3: track 0.00 -> 2.77 mm
- net GND: track 0.00 -> 2.70 mm
Other:
- board size 50 x 70 mm -> 50 x 40 mm

Commit message: User interface fix
Parts:
- moved L3002 10.7 mm to (101.3, 53.7), turned to -90 degrees
- moved L3001 10.1 mm to (88.5, 53.8), turned to -90 degrees
- moved TP3002 9.41 mm to (104.0, 62.0), turned to 0 degrees
- moved TP3001 8.49 mm to (88.5, 57.8), turned to 0 degrees
- moved C3002 8.10 mm to (96.8, 53.0), turned to -90 degrees
- moved C3005 5.86 mm to (104.3, 51.3), turned to 180 degrees
- moved C3008 5.55 mm to (104.5, 59.4), turned to 0 degrees
- moved C3006 5.30 mm to (108.0, 53.8), turned to 90 degrees
- moved U3001 5.22 mm to (93.5, 52.5)
- moved C3001 5.15 mm to (90.8, 53.0)
- moved C3004 3.01 mm to (92.0, 57.2), turned to 0 degrees
- moved C3007 2.66 mm to (104.5, 57.3), turned to 0 degrees
- moved U3002 2.08 mm to (104.8, 54.0), turned to 90 degrees
- moved C3003 0.25 mm to (92.0, 55.2), turned to 0 degrees

Commit message: LED module go brrrrrrrrrrrrrrrrrr
Parts:
- D501: renamed from D5001; moved to B.Cu
- D502: renamed from D5002; moved to B.Cu
- D503: renamed from D5003; moved to B.Cu
- D504: renamed from D5004; moved to B.Cu
- D505: renamed from D5005; moved to B.Cu
- D506: renamed from D5006; footprint LED_SMD:LED_PLCC_2835 -> footprints:JE2835_Amber; moved to B.Cu
- D507: renamed from D5007; footprint LED_SMD:LED_PLCC_2835 -> footprints:JE2835_Amber; moved to B.Cu
- D508: renamed from D5008; footprint LED_SMD:LED_PLCC_2835 -> footprints:JE2835_Amber; moved to B.Cu
- D509: renamed from D5009; footprint LED_SMD:LED_PLCC_2835 -> footprints:JE2835_Amber; moved to B.Cu
- L502: renamed from L5002; footprint Inductor_SMD:L_TDK_VLS6045EX_VLS6045AF -> Inductor_SMD:L_Coilcraft_XAL4040-XXX
- L503: renamed from L5003; footprint Inductor_SMD:L_Changjiang_FNR5045S -> Inductor_SMD:L_Sunlord_SWPA252012S
- Y401: renamed from Y4001; value Crystal -> 12M
- moved D505 194.4 mm to (92.0, 100.8), turned to 90 degrees
- moved D501 180.4 mm to (93.3, 90.0), turned to -90 degrees
- moved U501 167.8 mm to (91.3, 96.8), turned to 180 degrees
- moved TP504 164.5 mm to (88.8, 101.2)
- moved D504 160.2 mm to (123.0, 100.8), turned to 90 degrees
- moved R502 159.7 mm to (88.8, 96.8), turned to 90 degrees
- moved L501 158.2 mm to (95.6, 96.8)
- moved D509 158.2 mm to (88.0, 103.5), turned to 180 degrees
- moved L502 157.6 mm to (106.3, 101.5), turned to 180 degrees
- moved D508 155.2 mm to (88.1, 87.0), turned to 180 degrees
- moved D503 153.4 mm to (124.3, 90.0), turned to -90 degrees
- moved TP501 153.1 mm to (97.5, 101.2)
- moved D502 151.9 mm to (110.7, 94.9), turned to 180 degrees
- moved C501 151.6 mm to (90.2, 93.2), turned to 180 degrees
- moved C502 150.8 mm to (91.5, 95.0), turned to 180 degrees
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- renumbered C2001 to C201, C2002 to C202, C2003 to C203, C2004 to C204, C2005 to C205, C2006 to C206, C3001 to C301, C3002 to C302, C3003 to C303, C3004 to C304, C3005 to C305, C3006 to C306, C3007 to C307, C3008 to C308, C4001 to C401, C4002 to C402, C4003 to C403, C4004 to C404, C4005 to C405, C4006 to C406, C4007 to C407, C4008 to C408, C4009 to C409, C4010 to C410, C4011 to C411, C4012 to C412, C4013 to C413, C4014 to C414, C4015 to C415, C5001 to C501, C5002 to C502, C5003 to C503, C5004 to C504, C5005 to C505, C5006 to C506, C5007 to C507, C5008 to C508, C5009 to C509, C5010 to C510, C5011 to C511, C5012 to C512, C5013 to C513, C6001 to C601, C6002 to C602, D4001 to D401, D6001 to D601, D6002 to D602, D6003 to D603, F2001 to F201, J2001 to J201, J2002 to J202, J4001 to J401, J4002 to J402, JP2001 to JP201, L3001 to L301, L3002 to L302, L5001 to L501, R2001 to R201, R2002 to R202, R2003 to R203, R2004 to R204, R2005 to R205, R4001 to R401, R4002 to R402, R4003 to R403, R4004 to R404, R4005 to R405, R4006 to R406, R4007 to R407, R5001 to R501, R5002 to R502, R5003 to R503, R6001 to R601, R6002 to R602, R6003 to R603, R6004 to R604, R6005 to R605, SW4001 to SW401, SW4002 to SW402, TP2001 to TP201, TP3001 to TP301, TP3002 to TP302, TP5001 to TP501, TP5002 to TP502, TP5003 to TP503, TP5004 to TP504, TP5005 to TP505, TP5006 to TP506, U2001 to U201, U2002 to U202, U3001 to U301, U3002 to U302, U4001 to U401, U4002 to U402, U5001 to U501, U5002 to U502, U5003 to U503, U5004 to U504, U6001 to U601, U6002 to U602, Y2001 to Y201
Connections:
- C205 pad 2: Net-(U2002-OSC2) -> Net-(U202-OSC2)
- U202 pad 8: Net-(U2002-OSC2) -> Net-(U202-OSC2)
- U402 pad 38: /Microcontroller/GPIO26_ADC0 -> /LED_TEMP
- U504 pad 3: /LED_driver/LED_TEMP -> /LED_TEMP
- Y201 pad 3: GND -> Net-(U202-OSC2)
- Y201 pad 4: Net-(U2002-OSC2) -> GND
Routing:
- net /CAN_bus/CANH: track 0.00 -> 37.4 mm
- net /CAN_bus/CANL: track 0.00 -> 36.2 mm
- net /~{CS}: track 0.00 -> 27.9 mm, vias 0 -> 2
- net /MOSI: track 0.00 -> 27.8 mm, vias 0 -> 2
- net /MISO: track 0.00 -> 26.5 mm, vias 0 -> 2
- net /SCK: track 0.00 -> 26.1 mm, vias 0 -> 2
- net /Microcontroller/USB_D+: track 0.00 -> 22.1 mm
- net /Microcontroller/USB_D-: track 0.00 -> 21.5 mm
- net +3V3: track 2.77 -> 23.5 mm
- net /SCL: track 6.17 -> 24.1 mm, vias 0 -> 2
- net /SDA: track 5.03 -> 21.3 mm, vias 0 -> 2
- net /Microcontroller/~{RESET}: track 0.00 -> 13.5 mm
- net /Microcontroller/SWCLK: track 0.00 -> 12.1 mm, vias 0 -> 2
- net /Microcontroller/XIN: track 0.00 -> 10.7 mm
- net +5V: track 0.00 -> 10.7 mm
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- added copper zone on F.Cu, net +3V3
- added copper zone on F.Cu, net +5V
- added copper zone on F.Cu, net +SYSTEM
- added copper zone on F.Cu, net /PWM_AMBER
- added copper zone on F.Cu, net /PWM_RED
- added copper zone on F.Cu, net /PWM_WHITE
- added copper zone on F.Cu, net GND
- added copper zone on F.Cu, net Net-(D401-A)
- added copper zone on B.Cu, net Net-(D501-A)
- added copper zone on F.Cu, net Net-(D501-A)
- added copper zone on B.Cu, net Net-(D501-K)
- added copper zone on B.Cu, net Net-(D502-A)
- added copper zone on F.Cu, net Net-(D502-A)
- added copper zone on B.Cu, net Net-(D502-K)
- added copper zone on F.Cu, net Net-(D502-K)
- added copper zone on B.Cu, net Net-(D503-K)
- added copper zone on B.Cu, net Net-(D504-K)
- added copper zone on B.Cu, net Net-(D505-K)
- added copper zone on F.Cu, net Net-(D505-K)
- added copper zone on B.Cu, net Net-(D506-A)
- added copper zone on F.Cu, net Net-(D506-A)
- added copper zone on B.Cu, net Net-(D506-K)
- added copper zone on F.Cu, net Net-(D506-K)
- added copper zone on F.Cu, net Net-(F201-Pad1)
- added copper zone on F.Cu, net Net-(U301-SW)
- added copper zone on F.Cu, net Net-(U302-SW)
- added copper zone on F.Cu, net Net-(U501-SW)
- added copper zone on F.Cu, net Net-(U502-SW)
- added copper zone on F.Cu, net Net-(U503-SW)
Other:
- board size 50 x 40 mm -> 50 x 75.8 mm
- copper layers 2 -> 4

Commit message: User interface and Controller done
yes
Parts:
- added H101: MountingHole, MountingHole:MountingHole_3.2mm_M3, F.Cu at (87.0, 36.0)
- added H102: MountingHole, MountingHole:MountingHole_3.2mm_M3, F.Cu at (125.8, 46.0)
- added H103: MountingHole, MountingHole:MountingHole_3.2mm_M3, F.Cu at (86.8, 50.8)
- added H104: MountingHole, MountingHole:MountingHole_3.2mm_M3, F.Cu at (108.0, 66.0)
- C201, C202, C302, C306, C501, C503, C507, C508, C509, C512: footprint Capacitor_SMD:C_1206_3216Metric -> Capacitor_SMD:C_0805_2012Metric
- moved C513 34.0 mm to (110.2, 83.2), turned to -90 degrees
- moved U504 29.6 mm to (112.5, 83.2), turned to 180 degrees
- moved C501 4.00 mm to (90.2, 89.2)
- moved C502 4.00 mm to (91.5, 91.0)
- moved C503 4.00 mm to (111.3, 101.2)
- moved C504 4.00 mm to (110.1, 99.2)
- moved C505 4.00 mm to (91.8, 94.5)
- moved C506 4.00 mm to (109.8, 95.8)
- moved C507 4.00 mm to (96.0, 88.8)
- moved C508 4.00 mm to (106.5, 101.2)
- moved C509 4.00 mm to (122.7, 88.7)
- moved C510 4.00 mm to (125.6, 89.0)
- moved C511 4.00 mm to (126.2, 93.2)
- moved C512 4.00 mm to (128.4, 88.7)
- moved D501 4.00 mm to (93.3, 86.0)
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Routing:
- net /PWM_RED: track 0.00 -> 43.2 mm, vias 0 -> 4
- net /LED_TEMP: track 0.00 -> 42.5 mm, vias 0 -> 2
- net /PWM_WHITE: track 0.00 -> 39.9 mm, vias 0 -> 4
- net +5V: track 10.7 -> 46.9 mm, vias 0 -> 2
- net /PWM_AMBER: track 0.00 -> 36.0 mm, vias 0 -> 4
- net GND: track 3.70 -> 21.6 mm, vias 0 -> 196
- net +1V1: track 8.06 -> 23.5 mm, vias 0 -> 3
- net +3V3: track 23.5 -> 37.5 mm, vias 0 -> 24
- net Net-(U201-TXD): track 0.00 -> 8.08 mm
- net Net-(JP201-B): track 2.36 -> 5.54 mm
- net /SDA: track 21.3 -> 19.4 mm
- net /SCL: track 24.1 -> 22.5 mm
- net /Microcontroller/USB_D-: track 21.5 -> 22.3 mm
- net /Microcontroller/USB_D+: track 22.1 -> 22.9 mm
- net +SYSTEM: vias 0 -> 23
- added copper zone on In1.Cu, net +3V3
- added copper zone on In1.Cu, net +SYSTEM
- added copper zone on F.Cu, net /LED_TEMP
- added copper zone on B.Cu, net GND
- added copper zone on In2.Cu, net GND
- added copper zone on In2.Cu, net Net-(F201-Pad1)
Other:
- board size 50 x 75.8 mm -> 50 x 71.8 mm
- board text added: "3V3"
- board text added: "5V"
- board text added: "AMBER+"
- board text added: "AMBER-"
- board text added: "BOOT"
- board text added: "CAN TERM"
- board text added: "EENX16-VT24-27 LED Module"
- board text added: "RED+"
- board text added: "RED-"
- board text added: "RESET"
- board text added: "V_{in}"
- board text added: "WHITE+"
- board text added: "WHITE-"

Commit message: Changes and fixes
Parts:
- Y401: footprint Crystal:Crystal_SMD_Abracon_ABM3B-4Pin_5.0x3.2mm -> Crystal:Crystal_SMD_2520-4Pin_2.5x2.0mm
- moved C414 4.29 mm to (119.0, 64.4), turned to 90 degrees
- moved C415 2.18 mm to (123.4, 64.5), turned to -90 degrees
- moved Y401 1.45 mm to (121.3, 64.5), turned to 90 degrees
Routing:
- net /Microcontroller/XIN: track 10.8 -> 6.54 mm
- net GND: track 21.6 -> 20.6 mm, vias 196 -> 195
- net /Microcontroller/XOUT_R: track 3.94 -> 4.47 mm

Commit message: final fixes (hopefully) (GONE WRONG?!) (real)
Parts:
- moved F201 0.25 mm to (91.0, 44.5)
- moved H103 0.25 mm to (86.8, 50.5)
- moved C601 0.15 mm to (130.8, 44.2)
Routing:
- net GND: track 20.6 -> 17.1 mm, vias 195 -> 189
- net /CAN_bus/CANL: track 35.9 -> 37.1 mm
Other:
- board text added: "JLCJLCJLCJLC"
