File: Hardware/LED_Module/LED_Module.kicad_sch (KiCad schematic)
At the start: 0 parts

Commit message: La in allt
Myyycket saker
Other:
- sheet Sensors ports: added SCL, SDA, STATUS1, STATUS2, STATUS3; removed none
- company: (none) -> Chalmers EENX16-VT24-27

Commit message: LED module go brrrrrrrrrrrrrrrrrr
Other:
- sheet LED_driver ports: added LED_TEMP; removed none
Changed lines of the file:
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@@
+	(wire
+		(pts
+			(xy 95.25 93.98) (xy 96.52 93.98)
+		)
+		(stroke
+			(width 0)
+			(type default)
+		)
+	)
 	(wire
 		(pts
@@
 		(pts
 			(xy 95.25 72.39) (xy 96.52 72.39)
+		)
+		(stroke
+			(width 0)
+			(type default)
+		)
+	)
+	(wire
+		(pts
+			(xy 156.21 36.83) (xy 157.48 36.83)
 		)
 		(stroke
@@
 		)
 	)
+	(label "LED_TEMP"
+		(at 157.48 36.83 0)
+		(fields_autoplaced yes)
+		(effects
+			(font
+				(size 1.27 1.27)
+			)
+			(justify left bottom)
+		)
+	)
 	(label "~{CS}"
 		(at 129.54 58.42 180)
@@
 			)
 			(justify right bottom)
+		)
+	)
+	(label "LED_TEMP"
+		(at 96.52 93.98 0)
+		(fields_autoplaced yes)
+		(effects
+			(font
+				(size 1.27 1.27)
+			)
+			(justify left bottom)
 		)
 	)
@@
 			)
 		)
+		(pin "LED_TEMP" output
+			(at 156.21 36.83 0)
+			(effects
+				(font
+					(size 1.27 1.27)
+				)
+				(justify right)
+			)
+		)

Commit message: User interface and Controller done
yes
Parts:
- added H101, H102, H103, H104: MountingHole, MountingHole:MountingHole_3.2mm_M3, symbol Mechanical:MountingHole

Commit message: final fixes (hopefully) (GONE WRONG?!) (real)
Other:
- title: (none) -> Illumination system LED Module - overview
- moved on the sheet: H101, H102, H103, H104
