File: Hardware/LED_Module/LED_driver.kicad_sch (KiCad schematic)
At the start: 36 parts, among them U5 TPS92200, U8 TPS92200, U9 TPS92200

Commit message: La in allt
Myyycket saker
Parts:
- removed R11: 700m, symbol Device:R
- added C5013: 100n, Capacitor_SMD:C_0402_1005Metric, symbol Device:C
- added R5003: 200m, Resistor_SMD:R_1206_3216Metric, symbol Device:R
- added U5004: TMP236, Package_TO_SOT_SMD:SOT-353_SC-70-5, symbol Sensor_Temperature:TMP20AIDCK
- C5001: renamed from C25; footprint (none) -> Capacitor_SMD:C_1206_3216Metric; Footprint checked (none) -> YES; mouser (none) -> 581-1206DD106MAT2A
- C5002: renamed from C26; footprint (none) -> Capacitor_SMD:C_0402_1005Metric; Footprint checked (none) -> YES; REASON (none) -> GCM155R71H104KE02D is out of stock at RS; mouser (none) -> 81-GCM155R71H104KE2D
- C5003: renamed from C24; footprint (none) -> Capacitor_SMD:C_1206_3216Metric; Footprint checked (none) -> YES; mouser (none) -> 581-1206DD106MAT2A
- C5004: renamed from C23; footprint (none) -> Capacitor_SMD:C_0402_1005Metric; Footprint checked (none) -> YES; REASON (none) -> GCM155R71H104KE02D is out of stock at RS; mouser (none) -> 81-GCM155R71H104KE2D
- C5005: renamed from C27; footprint (none) -> Capacitor_SMD:C_0402_1005Metric; Footprint checked (none) -> YES; REASON (none) -> GCM155R71H104KE02D is out of stock at RS; mouser (none) -> 81-GCM155R71H104KE2D
- C5006: renamed from C22; footprint (none) -> Capacitor_SMD:C_0402_1005Metric; Footprint checked (none) -> YES; REASON (none) -> GCM155R71H104KE02D is out of stock at RS; mouser (none) -> 81-GCM155R71H104KE2D
- C5007: renamed from C28; footprint (none) -> Capacitor_SMD:C_1206_3216Metric; Footprint checked (none) -> YES; mouser (none) -> 581-1206DD106MAT2A
- C5008: renamed from C21; footprint (none) -> Capacitor_SMD:C_1206_3216Metric; Footprint checked (none) -> YES; mouser (none) -> 581-1206DD106MAT2A
- C5009: renamed from C29; footprint (none) -> Capacitor_SMD:C_1206_3216Metric; Footprint checked (none) -> YES; mouser (none) -> 581-1206DD106MAT2A
- C5010: renamed from C30; footprint (none) -> Capacitor_SMD:C_0402_1005Metric; Footprint checked (none) -> YES; REASON (none) -> GCM155R71H104KE02D is out of stock at RS; mouser (none) -> 81-GCM155R71H104KE2D
- C5011: renamed from C31; footprint (none) -> Capacitor_SMD:C_0402_1005Metric; Footprint checked (none) -> YES; REASON (none) -> GCM155R71H104KE02D is out of stock at RS; mouser (none) -> 81-GCM155R71H104KE2D
- C5012: renamed from C32; footprint (none) -> Capacitor_SMD:C_1206_3216Metric; Footprint checked (none) -> YES; mouser (none) -> 581-1206DD106MAT2A
- D5001: renamed from D2; value LED -> LED-red; footprint (none) -> footprints:KR DMLQ32. 23; Footprint checked (none) -> CHECKPOLARITY; mouser (none) -> 720-KRDMLQ32236K6M26
- D5002: renamed from D1; footprint (none) -> footprints:LUXEON 7070; Footprint checked (none) -> CHECKPOLARITY; mouser (none) -> 997-L1703070701200
- D5003: renamed from D3; value LED -> LED-red; footprint (none) -> footprints:KR DMLQ32. 23; Footprint checked (none) -> CHECKPOLARITY; mouser (none) -> 720-KRDMLQ32236K6M26
- D5004: renamed from D4; value LED -> LED-red; footprint (none) -> footprints:KR DMLQ32. 23; Footprint checked (none) -> CHECKPOLARITY; mouser (none) -> 720-KRDMLQ32236K6M26
- D5005: renamed from D5; value LED -> LED-red; footprint (none) -> footprints:KR DMLQ32. 23; Footprint checked (none) -> CHECKPOLARITY; mouser (none) -> 720-KRDMLQ32236K6M26
- D5006: renamed from D6; value LED -> LED-amber; footprint (none) -> LED_SMD:LED_PLCC_2835; Footprint checked (none) -> YES; mouser (none) -> 941-JE2835AAMN01AN
- D5007: renamed from D7; value LED -> LED-amber; footprint (none) -> LED_SMD:LED_PLCC_2835; Footprint checked (none) -> YES; mouser (none) -> 941-JE2835AAMN01AN
- D5008: renamed from D8; value LED -> LED-amber; footprint (none) -> LED_SMD:LED_PLCC_2835; Footprint checked (none) -> YES; mouser (none) -> 941-JE2835AAMN01AN
- D5009: renamed from D9; value LED -> LED-amber; footprint (none) -> LED_SMD:LED_PLCC_2835; Footprint checked (none) -> YES; mouser (none) -> 941-JE2835AAMN01AN
- L5001: renamed from L2; value 15u -> 20u; footprint (none) -> Inductor_SMD:L_Changjiang_FNR5045S; Footprint checked (none) -> YES; mouser (none) -> 810-VLS5045EX-220M
- L5002: renamed from L1; footprint (none) -> Inductor_SMD:L_TDK_VLS6045EX_VLS6045AF; Footprint checked (none) -> YES; mouser (none) -> 810-VLS6045EX-150M-H
- L5003: renamed from L3; value 100u -> 5.6u; footprint (none) -> Inductor_SMD:L_Changjiang_FNR5045S; Footprint checked (none) -> YES; mouser (none) -> 810-VLS5045EX-101M
- R5001: renamed from R9; footprint (none) -> Resistor_SMD:R_0805_2012Metric; Footprint checked (none) -> YES; mouser (none) -> 71-RCWE0805R100FKEA
- R5002: renamed from R10; footprint (none) -> Resistor_SMD:R_1206_3216Metric; Footprint checked (none) -> YES; mouser (none) -> 71-RCWE1206R200FKEA
- TP5001: renamed from TP6; footprint (none) -> TestPoint:TestPoint_Pad_D2.0mm; Footprint checked (none) -> YES
- TP5002: renamed from TP4; footprint (none) -> TestPoint:TestPoint_Pad_D2.0mm; Footprint checked (none) -> YES
- TP5003: renamed from TP5; footprint (none) -> TestPoint:TestPoint_Pad_D2.0mm; Footprint checked (none) -> YES
- TP5004: renamed from TP7; footprint (none) -> TestPoint:TestPoint_Pad_D2.0mm; Footprint checked (none) -> YES
- TP5005: renamed from TP9; footprint (none) -> TestPoint:TestPoint_Pad_D2.0mm; Footprint checked (none) -> YES
- TP5006: renamed from TP8; footprint (none) -> TestPoint:TestPoint_Pad_D2.0mm; Footprint checked (none) -> YES
- U5001: renamed from U8; Footprint checked (none) -> YES; REASON (none) -> TPS92200D1RXLR is not sold at RS or elfa; mouser (none) -> 595-TPS92200D1RXLR
- U5002: renamed from U5; Footprint checked (none) -> YES; REASON (none) -> TPS92200D1RXLR is not sold at RS or elfa; mouser (none) -> 595-TPS92200D1RXLR
- U5003: renamed from U9; Footprint checked (none) -> YES; REASON (none) -> TPS92200D1RXLR is not sold at RS or elfa; mouser (none) -> 595-TPS92200D1RXLR
Connections:
- net GND: now also C5013.2, R5003.2, U5004.2 (GND), U5004.5 (GND)
- net at D5007.1 (K): now also D5006.1 (K), D5008.1 (K), D5009.1 (K), TP5006.1, U5003.6 (FB), R5003.1; no longer D5008.2 (A)
- net at D5007.2 (A): now also C5012.1, D5006.2 (A), D5008.2 (A), D5009.2 (A), L5003.2, TP5005.1; no longer D5006.1 (K)
- net +BATT renamed +SYSTEM
- new net +3V3: C5013.1, U5004.4 (V_{DD})
- new net LED_TEMP: U5004.3 (V_{OUT})
Other:
- note added: "~0.75A peak"
- note added: "~1.5A peak"
- note added: "~1A peak"
- note removed: "~1.5A RMS ~1.5A peak"
- company: (none) -> Chalmers EENX16-VT24-27
- title: (none) -> LED's and drivers
- moved on the sheet: C5001, C5002, C5003, C5004, C5005, C5006, C5007, C5008, C5009, C5010, C5011, C5012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

Commit message: User interface fix
Parts:
- renumbered C5001 to C501, C5002 to C502, C5003 to C503, C5004 to C504, C5005 to C505, C5006 to C506, C5007 to C507, C5008 to C508, C5009 to C509, C5010 to C510, C5011 to C511, C5012 to C512, C5013 to C513, D5001 to D501, D5002 to D502, D5003 to D503, D5004 to D504, D5005 to D505, D5006 to D506, D5007 to D507, D5008 to D508, D5009 to D509, L5001 to L501, L5002 to L502, L5003 to L503, R5001 to R501, R5002 to R502, R5003 to R503, TP5001 to TP501, TP5002 to TP502, TP5003 to TP503, TP5004 to TP504, TP5005 to TP505, TP5006 to TP506, U5001 to U501, U5002 to U502, U5003 to U503, U5004 to U504

Commit message: LED module go brrrrrrrrrrrrrrrrrr
Parts:
- D506, D507, D508, D509: footprint LED_SMD:LED_PLCC_2835 -> footprints:JE2835_Amber
- L502: footprint Inductor_SMD:L_TDK_VLS6045EX_VLS6045AF -> Inductor_SMD:L_Coilcraft_XAL4040-XXX; mouser 810-VLS6045EX-150M-H -> 994-XAL4040-153MEC
- L503: footprint Inductor_SMD:L_Changjiang_FNR5045S -> Inductor_SMD:L_Sunlord_SWPA252012S; mouser 810-VLS5045EX-101M -> 520-MPI2520R1-5R6-R
Changed lines of the file:
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@@
 			)
 		)
-		(property "Footprint" "LED_SMD:LED_PLCC_2835"
+		(property "Footprint" "footprints:JE2835_Amber"
 			(at 105.41 120.65 0)
 			(effects
@@
 			)
 		)
-		(property "Footprint" "Inductor_SMD:L_Changjiang_FNR5045S"
+		(property "Footprint" "Inductor_SMD:L_Sunlord_SWPA252012S"
 			(at 76.2 107.95 0)
 			(effects
@@
 			)
 		)
-		(property "Datasheet" "https://product.tdk.com/system/files/dam/doc/product/inductor/inductor/smd/catalog/inductor_commercial_power_vls5045ex_en.pdf"
+		(property "Datasheet" "https://www.mouser.se/datasheet/2/122/ECS_MPI2520_SMD_POWER_INDUCTOR-1221975.pdf"
 			(at 76.2 107.95 0)
 			(effects
@@
 			)
 		)
-		(property "mouser" "810-VLS5045EX-101M"
+		(property "mouser" "520-MPI2520R1-5R6-R"
 			(at 76.2 107.95 90)
 			(effects
@@
 			)
 		)
-		(property "Footprint" "LED_SMD:LED_PLCC_2835"
+		(property "Footprint" "footprints:JE2835_Amber"
 			(at 121.92 120.65 0)
 			(effects
@@
 			)
 		)
-		(property "Footprint" "LED_SMD:LED_PLCC_2835"
+		(property "Footprint" "footprints:JE2835_Amber"
 			(at 88.9 120.65 0)
 			(effects
@@
 			)
 		)
-		(property "Footprint" "Inductor_SMD:L_TDK_VLS6045EX_VLS6045AF"
+		(property "Footprint" "Inductor_SMD:L_Coilcraft_XAL4040-XXX"
 			(at 168.91 38.1 0)
 			(effects
@@
 			)
 		)
-		(property "Datasheet" "https://product.tdk.com/system/files/dam/doc/product/inductor/inductor/smd/catalog/inductor_automotive_power_vls6045ex-h_en.pdf?ref_disty=mouser"
+		(property "Datasheet" "https://www.mouser.se/datasheet/2/597/xal4000-270751.pdf"
 			(at 168.91 38.1 0)
 			(effects
@@
 			)
 		)
-		(property "mouser" "810-VLS6045EX-150M-H"
+		(property "mouser" " 994-XAL4040-153MEC "
 			(at 168.91 38.1 0)
 			(effects
@@
 			)
 		)
-		(property "Footprint" "LED_SMD:LED_PLCC_2835"
+		(property "Footprint" "footprints:JE2835_Amber"
 			(at 138.43 120.65 0)
 			(effects

Commit message: User interface and Controller done
yes
Parts:
- C501, C503, C507, C508, C509, C512: footprint Capacitor_SMD:C_1206_3216Metric -> Capacitor_SMD:C_0805_2012Metric; mouser 581-1206DD106MAT2A -> 81-GRM21BR61H106KE3L
Changed lines of the file:
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@@
 			)
 		)
-		(property "Footprint" "Capacitor_SMD:C_1206_3216Metric"
+		(property "Footprint" "Capacitor_SMD:C_0805_2012Metric"
 			(at 80.9752 116.84 0)
 			(effects
@@
 			)
 		)
-		(property "Datasheet" "https://www.mouser.se/datasheet/2/40/cx5r_KGM-3223198.pdf"
+		(property "Datasheet" ""
 			(at 80.01 113.03 0)
 			(effects
@@
 			)
 		)
-		(property "mouser" "581-1206DD106MAT2A"
+		(property "mouser" "81-GRM21BR61H106KE3L"
 			(at 80.01 113.03 0)
 			(effects
@@
 			)
 		)
-		(property "Footprint" "Capacitor_SMD:C_1206_3216Metric"
+		(property "Footprint" "Capacitor_SMD:C_0805_2012Metric"
 			(at 25.0952 33.02 0)
 			(effects
@@
 			)
 		)
-		(property "Datasheet" "https://www.mouser.se/datasheet/2/40/cx5r_KGM-3223198.pdf"
+		(property "Datasheet" ""
 			(at 24.13 29.21 0)
 			(effects
@@
 			)
 		)
-		(property "mouser" "581-1206DD106MAT2A"
+		(property "mouser" "81-GRM21BR61H106KE3L"
 			(at 24.13 29.21 0)
 			(effects
@@
 			)
 		)
-		(property "Footprint" "Capacitor_SMD:C_1206_3216Metric"
+		(property "Footprint" "Capacitor_SMD:C_0805_2012Metric"
 			(at 25.0952 102.87 0)
 			(effects
@@
 			)
 		)
-		(property "Datasheet" "https://www.mouser.se/datasheet/2/40/cx5r_KGM-3223198.pdf"
+		(property "Datasheet" ""
 			(at 24.13 99.06 0)
 			(effects
@@
 			)
 		)
-		(property "mouser" "581-1206DD106MAT2A"
+		(property "mouser" "81-GRM21BR61H106KE3L"
 			(at 24.13 99.06 0)
 			(effects
@@
 			)
 		)
-		(property "Footprint" "Capacitor_SMD:C_1206_3216Metric"
+		(property "Footprint" "Capacitor_SMD:C_0805_2012Metric"
 			(at 80.9752 45.72 0)
 			(effects
@@
 			)
 		)
-		(property "Datasheet" "https://www.mouser.se/datasheet/2/40/cx5r_KGM-3223198.pdf"
+		(property "Datasheet" ""
 			(at 80.01 41.91 0)
 			(effects
@@
 			)
 		)
-		(property "mouser" "581-1206DD106MAT2A"
+		(property "mouser" "81-GRM21BR61H106KE3L"
 			(at 80.01 41.91 0)
 			(effects
@@
 			)
 		)
-		(property "Footprint" "Capacitor_SMD:C_1206_3216Metric"
+		(property "Footprint" "Capacitor_SMD:C_0805_2012Metric"
 			(at 173.6852 45.72 0)
 			(effects
@@
 			)
 		)
-		(property "Datasheet" "https://www.mouser.se/datasheet/2/40/cx5r_KGM-3223198.pdf"
+		(property "Datasheet" ""
 			(at 172.72 41.91 0)
 			(effects
@@
 			)
 		)
-		(property "mouser" "581-1206DD106MAT2A"
+		(property "mouser" "81-GRM21BR61H106KE3L"
 			(at 172.72 41.91 0)
 			(effects
@@
 			)
 		)
-		(property "Footprint" "Capacitor_SMD:C_1206_3216Metric"
+		(property "Footprint" "Capacitor_SMD:C_0805_2012Metric"
 			(at 117.8052 33.02 0)
 			(effects
@@
 			)
 		)
-		(property "Datasheet" "https://www.mouser.se/datasheet/2/40/cx5r_KGM-3223198.pdf"
+		(property "Datasheet" ""
 			(at 116.84 29.21 0)
 			(effects
@@
 			)
 		)
-		(property "mouser" "581-1206DD106MAT2A"
+		(property "mouser" "81-GRM21BR61H106KE3L"
 			(at 116.84 29.21 0)
 			(effects
