File: Hardware/LED_Module/Power.kicad_sch (KiCad schematic)
At the start: 18 parts, among them U10 AP63203WU, U11 AP63205WU

Commit message: La in allt
Myyycket saker
Parts:
- removed C33, C34, C35, C36, C38, C39, C41, C42: 10u, symbol Device:C
- removed C37, C40: 100n, symbol Device:C_Small
- removed F1: 4A, symbol Device:Fuse
- removed L4, L5: 4u7, symbol Device:L
- removed TP1: TP3V3, symbol Connector:TestPoint
- removed TP2: TP5V, symbol Connector:TestPoint
- removed TP3: TPVin, symbol Connector:TestPoint
- removed U10: AP63203WU, Package_TO_SOT_SMD:TSOT-23-6, symbol Regulator_Switching:AP63203WU
- removed U11: AP63205WU, Package_TO_SOT_SMD:TSOT-23-6, symbol Regulator_Switching:AP63205WU
- added C3001, C3005: 100n, Capacitor_SMD:C_0402_1005Metric, symbol Device:C_Small
- added C3002, C3006: 10u, Capacitor_SMD:C_1206_3216Metric, symbol Device:C
- added C3003, C3004, C3007, C3008: 22u, Capacitor_SMD:C_0805_2012Metric, symbol Device:C
- added L3001, L3002: 4u7, Inductor_SMD:L_1210_3225Metric, symbol Device:L
- added TP3001: TP3V3, TestPoint:TestPoint_Pad_D2.0mm, symbol Connector:TestPoint
- added TP3002: TP5V, TestPoint:TestPoint_Pad_D2.0mm, symbol Connector:TestPoint
- added U3001: AP63203WU, Package_TO_SOT_SMD:TSOT-23-6, symbol Regulator_Switching:AP63203WU
- added U3002: AP63205WU, Package_TO_SOT_SMD:TSOT-23-6, symbol Regulator_Switching:AP63205WU
Connections:
- net +3V3: now also C3003.1, C3004.1, L3001.2, TP3001.1, U3001.1 (FB)
- net +5V: now also C3002.1, C3007.1, C3008.1, L3002.2, TP3002.1, U3001.2 (EN), U3001.3 (IN), U3002.1 (FB)
- net GND: now also C3002.2, C3003.2, C3004.2, C3006.2, C3007.2, C3008.2, U3001.4 (GND), U3002.4 (GND)
- new net: C3005.1, L3002.1, U3002.5 (SW)
- new net: C3005.2, U3002.6 (BST)
- new net: C3001.1, L3001.1, U3001.5 (SW)
- new net: C3001.2, U3001.6 (BST)
- new net +SYSTEM: C3006.1, U3002.2 (EN), U3002.3 (IN)
Other:
- company: (none) -> Chalmers EENX16-VT24-27

Commit message: User interface fix
Parts:
- renumbered C3001 to C301, C3002 to C302, C3003 to C303, C3004 to C304, C3005 to C305, C3006 to C306, C3007 to C307, C3008 to C308, L3001 to L301, L3002 to L302, TP3001 to TP301, TP3002 to TP302, U3001 to U301, U3002 to U302
Changed lines of the file:
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@@
 		(dnp no)
 		(fields_autoplaced yes)
-		(property "Reference" "#PWR03002"
+		(property "Reference" "#PWR0302"
 			(at 101.6 48.26 0)
 			(effects
@@
 			(project "LED_Module"
 				(path "/16808901-367a-4ed1-b5c3-f1221533388f/ac7ce9ab-1b69-43a5-a489-e20382a6a58b"
-					(reference "#PWR03002")
+					(reference "#PWR0302")
 					(unit 1)
 				)
@@
 		(dnp no)
 		(fields_autoplaced yes)
-		(property "Reference" "C3005"
+		(property "Reference" "C305"
 			(at 77.47 96.5262 0)
 			(effects
@@
 			(project "LED_Module"
 				(path "/16808901-367a-4ed1-b5c3-f1221533388f/ac7ce9ab-1b69-43a5-a489-e20382a6a58b"
-					(reference "C3005")
+					(reference "C305")
 					(unit 1)
 				)
@@
 		(dnp no)
 		(fields_autoplaced yes)
-		(property "Reference" "#PWR03006"
+		(property "Reference" "#PWR0306"
 			(at 36.83 96.52 0)
 			(effects
@@
 			(project "LED_Module"
 				(path "/16808901-367a-4ed1-b5c3-f1221533388f/ac7ce9ab-1b69-43a5-a489-e20382a6a58b"
-					(reference "#PWR03006")
+					(reference "#PWR0306")
 					(unit 1)
 				)
@@
 		(on_board yes)
 		(dnp no)
-		(property "Reference" "C3008"
+		(property "Reference" "C308"
 			(at 101.854 97.028 0)
 			(effects
@@
 			(project "LED_Module"
 				(path "/16808901-367a-4ed1-b5c3-f1221533388f/ac7ce9ab-1b69-43a5-a489-e20382a6a58b"
-					(reference "C3008")
+					(reference "C308")
 					(unit 1)
 				)
@@
 		(on_board yes)
 		(dnp no)
-		(property "Reference" "C3006"
+		(property "Reference" "C306"
 			(at 37.084 97.028 0)
 			(effects
@@
 			(project "LED_Module"
 				(path "/16808901-367a-4ed1-b5c3-f1221533388f/ac7ce9ab-1b69-43a5-a489-e20382a6a58b"
-					(reference "C3006")
+					(reference "C306")
 					(unit 1)
 				)
@@
 		(on_board yes)
 		(dnp no)
-		(property "Reference" "TP3001"
+		(property "Reference" "TP301"
 			(at 93.98 35.814 0)
 			(effects
@@
 			(project "LED_Module"
 				(path "/16808901-367a-4ed1-b5c3-f1221533388f/ac7ce9ab-1b69-43a5-a489-e20382a6a58b"
-					(reference "TP3001")
+					(reference "TP301")
 					(unit 1)
 				)
@@
 		(dnp no)
 		(fields_autoplaced yes)
-		(property "Reference" "#PWR03010"
+		(property "Reference" "#PWR0310"
 			(at 55.88 111.76 0)
 			(effects
@@
 			(project "LED_Module"
 				(path "/16808901-367a-4ed1-b5c3-f1221533388f/ac7ce9ab-1b69-43a5-a489-e20382a6a58b"
-					(reference "#PWR03010")
+					(reference "#PWR0310")
 					(unit 1)
 				)
@@
 		(dnp no)
 		(fields_autoplaced yes)
-		(property "Reference" "#PWR03003"
+		(property "Reference" "#PWR0303"
 			(at 36.83 58.42 0)
 			(effects
@@
 			(project "LED_Module"
 				(path "/16808901-367a-4ed1-b5c3-f1221533388f/ac7ce9ab-1b69-43a5-a489-e20382a6a58b"
-					(reference "#PWR03003")
+					(reference "#PWR0303")
 					(unit 1)
 				)
@@
 		(dnp no)
 		(fields_autoplaced yes)
-		(property "Reference" "#PWR03007"
+		(property "Reference" "#PWR0307"
 			(at 101.6 99.06 0)
 			(effects
@@
 			(project "LED_Module"
 				(path "/16808901-367a-4ed1-b5c3-f1221533388f/ac7ce9ab-1b69-43a5-a489-e20382a6a58b"
-					(reference "#PWR03007")
+					(reference "#PWR0307")
 					(unit 1)
 				)
@@
 		(dnp no)
 		(fields_autoplaced yes)
-		(property "Reference" "L3001"
+		(property "Reference" "L301"
 			(at 78.74 39.37 90)
 			(effects
@@
 			(project "LED_Module"
 				(path "/16808901-367a-4ed1-b5c3-f1221533388f/ac7ce9ab-1b69-43a5-a489-e20382a6a58b"
-					(reference "L3001")
+					(reference "L301")
 					(unit 1)
 				)
@@
 		(dnp no)
 		(fields_autoplaced yes)
-		(property "Reference" "#PWR03005"
+		(property "Reference" "#PWR0305"
 			(at 55.88 60.96 0)
 			(effects
@@
 			(project "LED_Module"
 				(path "/16808901-367a-4ed1-b5c3-f1221533388f/ac7ce9ab-1b69-43a5-a489-e20382a6a58b"
-					(reference "#PWR03005")
+					(reference "#PWR0305")
 					(unit 1)
 				)
@@
 		(dnp no)
 		(fields_autoplaced yes)
-		(property "Reference" "U3002"
+		(property "Reference" "U302"
 			(at 55.88 87.63 0)
 			(effects
@@
 			(project "LED_Module"
 				(path "/16808901-367a-4ed1-b5c3-f1221533388f/ac7ce9ab-1b69-43a5-a489-e20382a6a58b"
-					(reference "U3002")
+					(reference "U302")
 					(unit 1)
 				)
@@
 		(dnp no)
 		(fields_autoplaced yes)
-		(property "Reference" "L3002"
+		(property "Reference" "L302"
 			(at 78.74 90.17 90)
 			(effects
@@
 			(project "LED_Module"
 				(path "/16808901-367a-4ed1-b5c3-f1221533388f/ac7ce9ab-1b69-43a5-a489-e20382a6a58b"
-					(reference "L3002")
+					(reference "L302")
 					(unit 1)
 				)
@@
 		(dnp no)
 		(fields_autoplaced yes)
-		(property "Reference" "#PWR03004"
+		(property "Reference" "#PWR0304"
 			(at 93.98 58.42 0)
 			(effects
@@
 			(project "LED_Module"
 				(path "/16808901-367a-4ed1-b5c3-f1221533388f/ac7ce9ab-1b69-43a5-a489-e20382a6a58b"
-					(reference "#PWR03004")
+					(reference "#PWR0304")
 					(unit 1)
 				)
@@
 		(dnp no)
 		(fields_autoplaced yes)
-		(property "Reference" "#PWR03008"
+		(property "Reference" "#PWR0308"
 			(at 36.83 109.22 0)
 			(effects
@@
 			(project "LED_Module"
 				(path "/16808901-367a-4ed1-b5c3-f1221533388f/ac7ce9ab-1b69-43a5-a489-e20382a6a58b"
-					(reference "#PWR03008")
+					(reference "#PWR0308")
 					(unit 1)
 				)
@@
 		(dnp no)
 		(fields_autoplaced yes)
-		(property "Reference" "#PWR03009"
+		(property "Reference" "#PWR0309"
 			(at 93.98 109.22 0)
 			(effects
@@
 			(project "LED_Module"
 				(path "/16808901-367a-4ed1-b5c3-f1221533388f/ac7ce9ab-1b69-43a5-a489-e20382a6a58b"
-					(reference "#PWR03009")
+					(reference "#PWR0309")
 					(unit 1)
 				)
@@
 		(on_board yes)
 		(dnp no)
-		(property "Reference" "C3002"
+		(property "Reference" "C302"
 			(at 37.084 46.228 0)
 			(effects
@@
 			(project "LED_Module"
 				(path "/16808901-367a-4ed1-b5c3-f1221533388f/ac7ce9ab-1b69-43a5-a489-e20382a6a58b"
-					(reference "C3002")
+					(reference "C302")
 					(unit 1)
 				)
@@
 		(dnp no)
 		(fields_autoplaced yes)
-		(property "Reference" "U3001"
+		(property "Reference" "U301"
 			(at 55.88 36.83 0)
 			(effects
@@
 			(project "LED_Module"
 				(path "/16808901-367a-4ed1-b5c3-f1221533388f/ac7ce9ab-1b69-43a5-a489-e20382a6a58b"
-					(reference "U3001")
+					(reference "U301")
 					(unit 1)
 				)
@@
 		(on_board yes)
 		(dnp no)
-		(property "Reference" "C3003"
+		(property "Reference" "C303"
 			(at 94.234 46.228 0)
 			(effects
@@
 			(project "LED_Module"
 				(path "/16808901-367a-4ed1-b5c3-f1221533388f/ac7ce9ab-1b69-43a5-a489-e20382a6a58b"
-					(reference "C3003")
+					(reference "C303")
 					(unit 1)
 				)
@@
 		(dnp no)
 		(fields_autoplaced yes)
-		(property "Reference" "C3001"
+		(property "Reference" "C301"
 			(at 77.47 45.7262 0)
 			(effects
@@
 			(project "LED_Module"
 				(path "/16808901-367a-4ed1-b5c3-f1221533388f/ac7ce9ab-1b69-43a5-a489-e20382a6a58b"
-					(reference "C3001")
+					(reference "C301")
 					(unit 1)
 				)
@@
 		(on_board yes)
 		(dnp no)
-		(property "Reference" "C3004"
+		(property "Reference" "C304"
 			(at 101.854 46.228 0)
 			(effects
@@
 			(project "LED_Module"
 				(path "/16808901-367a-4ed1-b5c3-f1221533388f/ac7ce9ab-1b69-43a5-a489-e20382a6a58b"
-					(reference "C3004")
+					(reference "C304")
 					(unit 1)
 				)
@@
 		(on_board yes)
 		(dnp no)
-		(property "Reference" "TP3002"
+		(property "Reference" "TP302"
 			(at 93.98 87.122 0)
 			(effects
@@
 			(project "LED_Module"
 				(path "/16808901-367a-4ed1-b5c3-f1221533388f/ac7ce9ab-1b69-43a5-a489-e20382a6a58b"
-					(reference "TP3002")
+					(reference "TP302")
 					(unit 1)
 				)
@@
 		(on_board yes)
 		(dnp no)
-		(property "Reference" "C3007"
+		(property "Reference" "C307"
 			(at 94.234 97.028 0)
 			(effects
@@
 			(project "LED_Module"
 				(path "/16808901-367a-4ed1-b5c3-f1221533388f/ac7ce9ab-1b69-43a5-a489-e20382a6a58b"
-					(reference "C3007")
+					(reference "C307")
 					(unit 1)
 				)
@@
 		(dnp no)
 		(fields_autoplaced yes)
-		(property "Reference" "#PWR03001"
+		(property "Reference" "#PWR0301"
 			(at 36.83 45.72 0)
 			(effects
@@
 			(project "LED_Module"
 				(path "/16808901-367a-4ed1-b5c3-f1221533388f/ac7ce9ab-1b69-43a5-a489-e20382a6a58b"
-					(reference "#PWR03001")
-					(unit 1)
-				)
+					(reference "#PWR0301")
+					(unit 1)
+				)

Commit message: User interface and Controller done
yes
Parts:
- C302, C306: footprint Capacitor_SMD:C_1206_3216Metric -> Capacitor_SMD:C_0805_2012Metric; mouser 581-1206DD106MAT2A -> 81-GRM21BR61H106KE3L
Changed lines of the file:
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@@
 			)
 		)
-		(property "Footprint" "Capacitor_SMD:C_1206_3216Metric"
+		(property "Footprint" "Capacitor_SMD:C_0805_2012Metric"
 			(at 37.7952 102.87 0)
 			(effects
@@
 			)
 		)
-		(property "Datasheet" "https://www.mouser.se/datasheet/2/40/cx5r_KGM-3223198.pdf"
+		(property "Datasheet" ""
 			(at 36.83 99.06 0)
 			(effects
@@
 			)
 		)
-		(property "mouser" "581-1206DD106MAT2A"
+		(property "mouser" "81-GRM21BR61H106KE3L"
 			(at 36.83 99.06 0)
 			(effects
@@
 			)
 		)
-		(property "Footprint" "Capacitor_SMD:C_1206_3216Metric"
+		(property "Footprint" "Capacitor_SMD:C_0805_2012Metric"
 			(at 37.7952 52.07 0)
 			(effects
@@
 			)
 		)
-		(property "Datasheet" "https://www.mouser.se/datasheet/2/40/cx5r_KGM-3223198.pdf"
+		(property "Datasheet" ""
 			(at 36.83 48.26 0)
 			(effects
@@
 			)
 		)
-		(property "mouser" "581-1206DD106MAT2A"
+		(property "mouser" "81-GRM21BR61H106KE3L"
 			(at 36.83 48.26 0)
 			(effects

Commit message: final fixes (hopefully) (GONE WRONG?!) (real)
Other:
- title: (none) -> Power Management - logic voltage regulators
Changed lines of the file:
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@@
 	(paper "A4")
 	(title_block
+		(title "Power Management - logic voltage regulators")
+		(date "2024-03-26")
+		(rev "B01")
 		(company "Chalmers EENX16-VT24-27")
 	)
