File: Hardware/LED_Module/Sensors.kicad_sch (KiCad schematic)
At the start: 12 parts, among them U3 LTR-303ALS-01, U4 MC3479

Commit message: La in allt
Myyycket saker
Parts:
- removed R16, R17: 4k7, symbol Device:R
- removed R18, R19, R20: 470, symbol Device:R
- added R6001, R6002: 5k1, Resistor_SMD:R_0402_1005Metric, symbol Device:R
- added R6003, R6004, R6005: 120, Resistor_SMD:R_0402_1005Metric, symbol Device:R
- C6001: renamed from C18; footprint (none) -> Capacitor_SMD:C_0402_1005Metric; Footprint checked (none) -> YES; REASON (none) -> GCM155R71H104KE02D is out of stock at RS; mouser (none) -> 81-GCM155R71H104KE2D
- C6002: renamed from C17; footprint (none) -> Capacitor_SMD:C_0402_1005Metric; Footprint checked (none) -> YES; REASON (none) -> GCM155R71H104KE02D is out of stock at RS; mouser (none) -> 81-GCM155R71H104KE2D
- D6001: renamed from D11; footprint (none) -> LED_SMD:LED_0603_1608Metric; Footprint checked (none) -> YES; mouser (none) -> 710-150060RS75003
- D6002: renamed from D12; footprint (none) -> LED_SMD:LED_0603_1608Metric; Footprint checked (none) -> YES; mouser (none) -> 710-150060GS75003
- D6003: renamed from D13; footprint (none) -> LED_SMD:LED_0603_1608Metric; Footprint checked (none) -> YES; mouser (none) -> 710-150060BS84000
- U6001: renamed from U4; Footprint checked (none) -> YES; REASON (none) -> MC3479 is not sold at RS or elfa; mouser (none) -> 498-MC3479
- U6002: renamed from U3; Footprint checked (none) -> YES; REASON (none) -> LTR-303ALS-01 is not sold at RS or elfa; mouser (none) -> 859-LTR-303ALS-01
Connections:
- net +3V3: now also R6001.1, R6002.1
- net GND: now also R6003.2, R6004.2, R6005.2
- net SCL: now also R6001.2
- net SDA: now also R6002.2
- net at D6003.1 (K): now also R6005.1
- net at D6002.1 (K): now also R6004.1
- net at D6001.1 (K): now also R6003.1
Other:
- company: (none) -> Chalmers EENX16-VT24-27
- moved on the sheet: D6002, D6003

Commit message: User interface fix
Parts:
- renumbered C6001 to C601, C6002 to C602, D6001 to D601, D6002 to D602, D6003 to D603, R6001 to R601, R6002 to R602, R6003 to R603, R6004 to R604, R6005 to R605, U6001 to U601, U6002 to U602
Changed lines of the file:
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@@
 		(dnp no)
 		(fields_autoplaced yes)
-		(property "Reference" "#PWR06001"
+		(property "Reference" "#PWR0601"
 			(at 41.91 27.94 0)
 			(effects
@@
 			(project "LED_Module"
 				(path "/16808901-367a-4ed1-b5c3-f1221533388f/e9010f9b-e0a7-41f4-995c-14b2e7b39a86"
-					(reference "#PWR06001")
+					(reference "#PWR0601")
 					(unit 1)
 				)
@@
 		(dnp no)
 		(fields_autoplaced yes)
-		(property "Reference" "D6003"
+		(property "Reference" "D603"
 			(at 63.5 62.5474 90)
 			(effects
@@
 			(project "LED_Module"
 				(path "/16808901-367a-4ed1-b5c3-f1221533388f/e9010f9b-e0a7-41f4-995c-14b2e7b39a86"
-					(reference "D6003")
+					(reference "D603")
 					(unit 1)
 				)
@@
 		(dnp no)
 		(fields_autoplaced yes)
-		(property "Reference" "D6002"
+		(property "Reference" "D602"
 			(at 52.07 62.5474 90)
 			(effects
@@
 			(project "LED_Module"
 				(path "/16808901-367a-4ed1-b5c3-f1221533388f/e9010f9b-e0a7-41f4-995c-14b2e7b39a86"
-					(reference "D6002")
+					(reference "D602")
 					(unit 1)
 				)
@@
 		(dnp no)
 		(fields_autoplaced yes)
-		(property "Reference" "#PWR06007"
+		(property "Reference" "#PWR0607"
 			(at 129.54 82.55 0)
 			(effects
@@
 			(project "LED_Module"
 				(path "/16808901-367a-4ed1-b5c3-f1221533388f/e9010f9b-e0a7-41f4-995c-14b2e7b39a86"
-					(reference "#PWR06007")
+					(reference "#PWR0607")
 					(unit 1)
 				)
@@
 		(dnp no)
 		(fields_autoplaced yes)
-		(property "Reference" "#PWR06009"
+		(property "Reference" "#PWR0609"
 			(at 106.68 97.79 0)
 			(effects
@@
 			(project "LED_Module"
 				(path "/16808901-367a-4ed1-b5c3-f1221533388f/e9010f9b-e0a7-41f4-995c-14b2e7b39a86"
-					(reference "#PWR06009")
+					(reference "#PWR0609")
 					(unit 1)
 				)
@@
 		(dnp no)
 		(fields_autoplaced yes)
-		(property "Reference" "C6001"
+		(property "Reference" "C601"
 			(at 147.32 30.4799 0)
 			(effects
@@
 			(project "LED_Module"
 				(path "/16808901-367a-4ed1-b5c3-f1221533388f/e9010f9b-e0a7-41f4-995c-14b2e7b39a86"
-					(reference "C6001")
+					(reference "C601")
 					(unit 1)
 				)
@@
 		(on_board yes)
 		(dnp no)
-		(property "Reference" "U6002"
+		(property "Reference" "U602"
 			(at 110.744 70.612 0)
 			(effects
@@
 			(project "LED_Module"
 				(path "/16808901-367a-4ed1-b5c3-f1221533388f/e9010f9b-e0a7-41f4-995c-14b2e7b39a86"
-					(reference "U6002")
+					(reference "U602")
 					(unit 1)
 				)
@@
 		(dnp no)
 		(fields_autoplaced yes)
-		(property "Reference" "#PWR06006"
+		(property "Reference" "#PWR0606"
 			(at 106.68 72.39 0)
 			(effects
@@
 			(project "LED_Module"
 				(path "/16808901-367a-4ed1-b5c3-f1221533388f/e9010f9b-e0a7-41f4-995c-14b2e7b39a86"
-					(reference "#PWR06006")
+					(reference "#PWR0606")
 					(unit 1)
 				)
@@
 		(dnp no)
 		(fields_autoplaced yes)
-		(property "Reference" "#PWR06005"
+		(property "Reference" "#PWR0605"
 			(at 111.76 58.42 0)
 			(effects
@@
 			(project "LED_Module"
 				(path "/16808901-367a-4ed1-b5c3-f1221533388f/e9010f9b-e0a7-41f4-995c-14b2e7b39a86"
-					(reference "#PWR06005")
+					(reference "#PWR0605")
 					(unit 1)
 				)
@@
 		(dnp no)
 		(fields_autoplaced yes)
-		(property "Reference" "D6001"
+		(property "Reference" "D601"
 			(at 40.64 62.5474 90)
 			(effects
@@
 			(project "LED_Module"
 				(path "/16808901-367a-4ed1-b5c3-f1221533388f/e9010f9b-e0a7-41f4-995c-14b2e7b39a86"
-					(reference "D6001")
+					(reference "D601")
 					(unit 1)
 				)
@@
 		(on_board yes)
 		(dnp no)
-		(property "Reference" "U6001"
+		(property "Reference" "U601"
 			(at 119.38 30.48 0)
 			(effects
@@
 			(project "LED_Module"
 				(path "/16808901-367a-4ed1-b5c3-f1221533388f/e9010f9b-e0a7-41f4-995c-14b2e7b39a86"
-					(reference "U6001")
+					(reference "U601")
 					(unit 1)
 				)
@@
 		(dnp no)
 		(fields_autoplaced yes)
-		(property "Reference" "R6003"
+		(property "Reference" "R603"
 			(at 39.37 71.1199 0)
 			(effects
@@
 			(project "LED_Module"
 				(path "/16808901-367a-4ed1-b5c3-f1221533388f/e9010f9b-e0a7-41f4-995c-14b2e7b39a86"
-					(reference "R6003")
+					(reference "R603")
 					(unit 1)
 				)
@@
 		(dnp no)
 		(fields_autoplaced yes)
-		(property "Reference" "#PWR06008"
+		(property "Reference" "#PWR0608"
 			(at 36.83 83.82 0)
 			(effects
@@
 			(project "LED_Module"
 				(path "/16808901-367a-4ed1-b5c3-f1221533388f/e9010f9b-e0a7-41f4-995c-14b2e7b39a86"
-					(reference "#PWR06008")
+					(reference "#PWR0608")
 					(unit 1)
 				)
@@
 		(dnp no)
 		(fields_autoplaced yes)
-		(property "Reference" "R6001"
+		(property "Reference" "R601"
 			(at 44.45 27.9399 0)
 			(effects
@@
 			(project "LED_Module"
 				(path "/16808901-367a-4ed1-b5c3-f1221533388f/e9010f9b-e0a7-41f4-995c-14b2e7b39a86"
-					(reference "R6001")
+					(reference "R601")
 					(unit 1)
 				)
@@
 		(dnp no)
 		(fields_autoplaced yes)
-		(property "Reference" "R6004"
+		(property "Reference" "R604"
 			(at 50.8 71.1199 0)
 			(effects
@@
 			(project "LED_Module"
 				(path "/16808901-367a-4ed1-b5c3-f1221533388f/e9010f9b-e0a7-41f4-995c-14b2e7b39a86"
-					(reference "R6004")
+					(reference "R604")
 					(unit 1)
 				)
@@
 		(dnp no)
 		(fields_autoplaced yes)
-		(property "Reference" "#PWR06002"
+		(property "Reference" "#PWR0602"
 			(at 113.03 31.75 0)
 			(effects
@@
 			(project "LED_Module"
 				(path "/16808901-367a-4ed1-b5c3-f1221533388f/e9010f9b-e0a7-41f4-995c-14b2e7b39a86"
-					(reference "#PWR06002")
+					(reference "#PWR0602")
 					(unit 1)
 				)
@@
 		(dnp no)
 		(fields_autoplaced yes)
-		(property "Reference" "#PWR06003"
+		(property "Reference" "#PWR0603"
 			(at 143.51 41.91 0)
 			(effects
@@
 			(project "LED_Module"
 				(path "/16808901-367a-4ed1-b5c3-f1221533388f/e9010f9b-e0a7-41f4-995c-14b2e7b39a86"
-					(reference "#PWR06003")
+					(reference "#PWR0603")
 					(unit 1)
 				)
@@
 		(dnp no)
 		(fields_autoplaced yes)
-		(property "Reference" "C6002"
+		(property "Reference" "C602"
 			(at 133.35 71.1199 0)
 			(effects
@@
 			(project "LED_Module"
 				(path "/16808901-367a-4ed1-b5c3-f1221533388f/e9010f9b-e0a7-41f4-995c-14b2e7b39a86"
-					(reference "C6002")
+					(reference "C602")
 					(unit 1)
 				)
@@
 		(dnp no)
 		(fields_autoplaced yes)
-		(property "Reference" "#PWR06004"
+		(property "Reference" "#PWR0604"
 			(at 95.25 54.61 0)
 			(effects
@@
 			(project "LED_Module"
 				(path "/16808901-367a-4ed1-b5c3-f1221533388f/e9010f9b-e0a7-41f4-995c-14b2e7b39a86"
-					(reference "#PWR06004")
+					(reference "#PWR0604")
 					(unit 1)
 				)
@@
 		(dnp no)
 		(fields_autoplaced yes)
-		(property "Reference" "R6002"
+		(property "Reference" "R602"
 			(at 54.61 27.9399 0)
 			(effects
@@
 			(project "LED_Module"
 				(path "/16808901-367a-4ed1-b5c3-f1221533388f/e9010f9b-e0a7-41f4-995c-14b2e7b39a86"
-					(reference "R6002")
+					(reference "R602")
 					(unit 1)
 				)
@@
 		(dnp no)
 		(fields_autoplaced yes)
-		(property "Reference" "R6005"
+		(property "Reference" "R605"
 			(at 62.23 71.1199 0)
 			(effects
@@
 			(project "LED_Module"
 				(path "/16808901-367a-4ed1-b5c3-f1221533388f/e9010f9b-e0a7-41f4-995c-14b2e7b39a86"
-					(reference "R6005")
+					(reference "R605")
 					(unit 1)
 				)

Commit message: final fixes (hopefully) (GONE WRONG?!) (real)
Other:
- title: (none) -> Sensors - accelerometer, ambient light and status LEDs
Changed lines of the file:
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@@
 	(paper "A4")
 	(title_block
+		(title "Sensors - accelerometer, ambient light and status LEDs")
+		(date "2024-03-26")
+		(rev "B01")
 		(company "Chalmers EENX16-VT24-27")
 	)
