File: Hardware/Controller/CAN_bus.kicad_sch (KiCad schematic)
At the start: 16 parts, among them J5 RJ10, J6 RJ10, Q2 Si7461DP, Q3 Q_NMOS_GSD, U2 MCP2515-xST, U6 MCP2551-I-SN, Y2 8M

Commit message: La in allt
Myyycket saker
Parts:
- added R5007: 5k1, Resistor_SMD:R_0402_1005Metric, symbol Device:R
- C5001: renamed from C45; value C -> 10p; footprint (none) -> Capacitor_SMD:C_0402_1005Metric; mouser (none) -> 81-GRT1555C2A100JA2J
- C5002: renamed from C46; value C -> 10p; footprint (none) -> Capacitor_SMD:C_0402_1005Metric; mouser (none) -> 81-GRT1555C2A100JA2J
- J5001: renamed from J5; value RJ10 -> RJ9; mouser (none) -> 649-61835-0441LF
- J5002: renamed from J6; value RJ10 -> RJ9; mouser (none) -> 649-61835-0441LF
- JP5001: renamed from JP1; footprint (none) -> Connector_PinHeader_2.54mm:PinHeader_1x02_P2.54mm_Vertical; ETA (none) -> ETA
- Q5001: renamed from Q2; mouser (none) -> 781-SI7461DP-T1-E3
- Q5002: renamed from Q3; ETA (none) -> ETA
- R5001: renamed from R34; footprint (none) -> Resistor_SMD:R_0402_1005Metric; mouser (none) -> 71-CRCW040210K0JNEDC
- R5002: renamed from R32; footprint (none) -> Resistor_SMD:R_0402_1005Metric; mouser (none) -> 71-CRCW0402120RFKED
- R5003: renamed from R29; value 5k -> 5k1; footprint (none) -> Resistor_SMD:R_0402_1005Metric; mouser (none) -> 71-CRCW0402-5.1K-E3
- R5004: renamed from R30; footprint (none) -> Resistor_SMD:R_0402_1005Metric; mouser (none) -> 71-CRCW040210K0JNEDC
- R5005: renamed from R31; footprint (none) -> Resistor_SMD:R_0402_1005Metric; mouser (none) -> 71-CRCW040210K0JNEDC
- R5006: renamed from R28; footprint (none) -> Resistor_SMD:R_0402_1005Metric; mouser (none) -> 71-CRCW040210K0JNEDC
- U5001: renamed from U6; ETA (none) -> ETA
- U5002: renamed from U2; ETA (none) -> ETA
- Y5001: renamed from Y2; footprint (none) -> Crystal:Crystal_SMD_Abracon_ABM3B-4Pin_5.0x3.2mm; mouser (none) -> 815-ABM3B8MHZ101UT
Connections:
- net at Q5001.4 (G), R5001.2: now also R5007.1; no longer Q5002.3 (D)
- net +BATT renamed +SYSTEM
- new net: Q5002.3 (D), R5007.2
Other:
- moved on the sheet: C5001, C5002, Q5002, R5001, R5006, U5002, Y5001

Commit message: User interface fix
Parts:
- renumbered C5001 to C501, C5002 to C502, J5001 to J501, J5002 to J502, JP5001 to JP501, Q5001 to Q501, Q5002 to Q502, R5001 to R501, R5007 to R502, R5002 to R503, R5003 to R504, R5004 to R505, R5005 to R506, R5006 to R507, U5001 to U501, U5002 to U502, Y5001 to Y501

Commit message: User interface and Controller done
yes
Parts:
- Y501: symbol Device:Crystal_GND23 -> Device:Crystal_GND24
Connections:
- net GND: now also Y501.4; no longer Y501.3
- net at C501.2, U502.8 (OSC2): now also Y501.3; no longer Y501.4
Changed lines of the file:
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@@
 	)
 	(symbol
-		(lib_id "Device:Crystal_GND23")
+		(lib_id "Device:Crystal_GND24")
 		(at 54.61 101.6 90)
 		(unit 1)
@@
 			)
 		)
-		(property "Datasheet" "https://www.mouser.se/datasheet/2/3/abm3b-1774998.pdf"
+		(property "Datasheet" "~"
 			(at 54.61 101.6 0)
 			(effects
@@
 			)
 		)
-		(property "Description" ""
+		(property "Description" "Four pin crystal, GND on pins 2 and 4"
 			(at 54.61 101.6 0)
 			(effects

Commit message: Changes and fixes
Parts:
- Q501: footprint Package_SO:Vishay_PowerPAK_1212-8_Single -> Package_SO:PowerPAK_SO-8_Single
Changed lines of the file:
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@@
 			)
 		)
-		(property "Footprint" "Package_SO:Vishay_PowerPAK_1212-8_Single"
+		(property "Footprint" "Package_SO:PowerPAK_SO-8_Single"
 			(at 209.55 43.815 0)
 			(effects
