File: Hardware/Controller/Battery.kicad_sch (KiCad schematic)
At the start: 34 parts, among them J3 XT60, Q2 PMOS, Q3 Q_Dual_NMOS_S1G1S2G2D2D2D1D1, Q4 NMOS, Q5 NMOS, Q6 NMOS, Q7 NMOS, U5 LTC4020

Commit message: Controller fixades
Parts:
- removed Q2: PMOS, symbol Simulation_SPICE:PMOS
- removed Q3: Q_Dual_NMOS_S1G1S2G2D2D2D1D1, Package_SO:Vishay_PowerPAK_1212-8_Dual, symbol Device:Q_Dual_NMOS_S1G1S2G2D2D2D1D1
- removed Q4, Q5, Q6, Q7: NMOS, symbol Simulation_SPICE:NMOS
- added C1: 1n, symbol Device:C_Small
- added C21, C23, C3, C31, C32, C33, C34, C35, C36, C37, C38, C47, C48, C51, C52, C53, C54: 10u, symbol Device:C
- added C39: 100n, symbol Device:C
- added C40: 33n, symbol Device:C
- added C41, C42, C43, C44: 56u, symbol Device:C_Polarized
- added C49, C50: 100n, symbol Device:C_Small
- added D1: BZX84C6V2L, Package_TO_SOT_SMD:SOT-23, symbol Diode:BZX84Cxx
- added F1: 5A, symbol Device:Fuse
- added F2: 10A, symbol Device:Fuse
- added J1: Conn_PTC, symbol Connector_Generic:Conn_01x02
- added L2, L3: 4u7, symbol Device:L
- added Q4, Q8: Si7960DP, Package_SO:Vishay_PowerPAK_1212-8_Dual, symbol symbols:Si7272DP
- added Q5: Si7461DP, Package_SO:Vishay_PowerPAK_1212-8_Single, symbol Transistor_FET:SiS415DNT
- added R1: 100, symbol Device:R
- added R2: 105k, symbol Device:R
- added R25: 10k, symbol Device:R
- added R33: 47k, symbol Device:R_Small
- added TH1: 10k NTC, symbol Device:Thermistor_NTC
- added TP1: TP3V3, symbol Connector:TestPoint
- added TP2: TP5V, symbol Connector:TestPoint
- added U7: AP63203WU, Package_TO_SOT_SMD:TSOT-23-6, symbol Regulator_Switching:AP63203WU
- added U8: AP63205WU, Package_TO_SOT_SMD:TSOT-23-6, symbol Regulator_Switching:AP63205WU
- C24: value C -> 10n
- C25: value C -> 680p
- C26: value C -> 68p
- C27: value C -> 100p
- D4, D5: value D_Schottky -> SBR0560S1
- R13: value RsenseA -> 8m
- R14: value RsenseB -> 8m
- R15, R16: value 2k7 -> 1k
- R18: value R -> 56k
- R19: value R -> 47k
- R20: value 2.5m -> 2m
- R21: value 68k -> 215k
- R22: value 10k -> 24k9
Connections:
- net +BATT: now also C47.1, C48.1, F1.2, R33.1, U7.2 (EN), U7.3 (IN), U8.3 (IN); no longer R20.4, R21.1
- net GND: now also C21.2, C23.2, C3.2, C31.2, C32.2, C33.2, C34.2, C35.2, C36.2, C37.2, C38.2, C39.2, C41.2, C42.2, C43.2, C44.2, C47.2, C48.2, C51.2, C52.2, C53.2, C54.2, J1.2 (Pin_2), R25.2, TH1.2, U7.4 (GND), U8.4 (GND); no longer C29.2, C30.2
- net INTVcc: now also C3.1; no longer R15.1, R16.1
- net VBUS: now also C21.1, C23.1, C31.1, C32.1, C33.1, C39.1, C41.1, C42.1, R2.1
- net SW1: now reaches L1.1, U5.38 (SW1)
- net SW1: now also Q8.1 (S), Q8.5 (D)
- net BG1: now reaches U5.37 (BG1)
- net BG1: now also Q8.4 (G)
- net at R14.4: now also Q4.3 (S), Q8.3 (S)
- net at R13.1: now also Q8.6 (D)
- net TG1: now reaches U5.1 (TG1)
- net TG1: now also C29.1, Q8.2 (G)
- net SENSTOP: now reaches R13.2, U5.6 (SENSTOP)
- net SENSVin: now reaches R13.3, U5.7 (SENSVin)
- net BST2: now reaches C30.1, D5.1 (K), U5.30 (BST2)
- net BST2: now also D1.3 (K)
- net CSP: now reaches C28.1, R23.1, U5.23 (CSP)
- net BST1: now reaches D4.1 (K), U5.2 (BST1)
- net BST1: now also C29.2; no longer C29.1
- net STAT1: now reaches D2.1 (K), U5.12 (STAT1)
- net STAT2: now reaches D3.1 (K), U5.13 (STAT2)
- net NTC: now reaches U5.16 (NTC)
- net NTC: now also J1.1 (Pin_1), TH1.1
- net BAT: now reaches R26.1, U5.20 (BAT)
- net BAT: now also F2.1, Q5.1 (S), Q5.2 (S), Q5.3 (S); no longer J3.2 (Pin_2)
- net BGATE: now reaches U5.21 (BGATE)
- net BGATE: now also C1.2, Q5.4 (G)
- net CSN: now reaches R24.2, U5.22 (CSN)
- net CSN: now also R1.1; no longer R20.2
- net TG2: now reaches U5.31 (TG2)
- net TG2: now also Q4.2 (G)
- net SW2: now reaches L1.2, U5.32 (SW2)
- net SW2: now also C30.2, D1.1 (A), Q4.1 (S), Q4.5 (D)
- net BG2: now reaches U5.33 (BG2)
- net BG2: now also Q4.4 (G)
- net SENSGND: now reaches R14.2, U5.4 (SENSGND)
- net SENSGND: now also C40.2
- net SENSBOT: now reaches R14.3, U5.5 (SENSBOT)
- net SENSBOT: now also C40.1
- net RT: now reaches R17.1, U5.8 (RT)
- net SHDN: now reaches U5.9 (SHDN)
- net SHDN: now also R2.2, R25.1
- net at R20.1: now also Q5.5 (D)
- new net: C1.1, R1.2, R20.2
- new net: C50.1, L3.1, U8.5 (SW)
- new net: C50.2, U8.6 (BST)
- new net: F2.2, J3.2 (Pin_2)
- new net: C49.1, L2.1, U7.5 (SW)
- new net: C49.2, U7.6 (BST)
- new net +3V3: C51.1, C53.1, L2.2, R15.1, R16.1, TP1.1, U7.1 (FB)
- new net +5V: C52.1, C54.1, L3.2, TP2.1, U8.1 (FB)
- new net 5V_EN: R33.2, U8.2 (EN)
- new net BATT_RAW: C34.1, C35.1, C36.1, C37.1, C38.1, C43.1, C44.1, F1.1, Q4.6 (D), R20.4, R21.1
Other:
- note added: "Connect through connector, couple thermally to the battery"
- company: (none) -> Chalmers EENX16-VT24-27
- title: (none) -> Battery charging and power management
- moved on the sheet: C24, C25, C26, C27, C28, C29, C30, D2, D3, D5, J3, R15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

Commit message: La in allt
Myyycket saker
Parts:
- removed C47, C48, C51, C52, C53, C54: 10u, symbol Device:C
- removed C49, C50: 100n, symbol Device:C_Small
- removed J3: XT60, symbol Connector_Generic:Conn_01x02
- removed L2, L3: 4u7, symbol Device:L
- removed R33: 47k, symbol Device:R_Small
- removed TP1: TP3V3, symbol Connector:TestPoint
- removed TP2: TP5V, symbol Connector:TestPoint
- removed U7: AP63203WU, Package_TO_SOT_SMD:TSOT-23-6, symbol Regulator_Switching:AP63203WU
- removed U8: AP63205WU, Package_TO_SOT_SMD:TSOT-23-6, symbol Regulator_Switching:AP63205WU
- added C4034, C4038: 100n, Capacitor_SMD:C_0402_1005Metric, symbol Device:C_Small
- added C4035, C4039: 10u, Capacitor_SMD:C_0805_2012Metric, symbol Device:C
- added C4036, C4037, C4040, C4041: 22u, Capacitor_SMD:C_0805_2012Metric, symbol Device:C
- added D4006: MBRS360, Diode_SMD:D_SMC, symbol Device:D_Schottky
- added J4001: Conn_balance, Connector_JST:JST_VH_B7P-VH-FB-B_1x07_P3.96mm_Vertical, symbol Connector:Conn_01x07_Socket
- added J4002: XT60, Connector_AMASS:AMASS_XT60IPW-M_1x03_P7.20mm_Horizontal, symbol Connector_Generic:Conn_01x02
- added L4004, L4005: 4u7, Inductor_SMD:L_1210_3225Metric, symbol Device:L
- added TP4003: BAT_UNPROT-, TestPoint:TestPoint_Pad_2.5x2.5mm, symbol Connector:TestPoint
- added TP4004: BAT_S5, TestPoint:TestPoint_Pad_2.5x2.5mm, symbol Connector:TestPoint
- added TP4005: BAT_S4, TestPoint:TestPoint_Pad_2.5x2.5mm, symbol Connector:TestPoint
- added TP4006: BAT_S3, TestPoint:TestPoint_Pad_2.5x2.5mm, symbol Connector:TestPoint
- added TP4007: BAT_S2, TestPoint:TestPoint_Pad_2.5x2.5mm, symbol Connector:TestPoint
- added TP4008: BAT_S1, TestPoint:TestPoint_Pad_2.5x2.5mm, symbol Connector:TestPoint
- added TP4009: BAT_UNPROT+, TestPoint:TestPoint_Pad_2.5x2.5mm, symbol Connector:TestPoint
- added TP4010: BAT_PROT+, TestPoint:TestPoint_Pad_2.5x2.5mm, symbol Connector:TestPoint
- added TP4011: BAT_PROT-, TestPoint:TestPoint_Pad_2.5x2.5mm, symbol Connector:TestPoint
- added TP4012: TP3V3, TestPoint:TestPoint_Pad_D2.0mm, symbol Connector:TestPoint
- added TP4013: TP5V, TestPoint:TestPoint_Pad_D2.0mm, symbol Connector:TestPoint
- added U4004: AP63203WU, Package_TO_SOT_SMD:TSOT-23-6, symbol Regulator_Switching:AP63203WU
- added U4005: AP63205WU, Package_TO_SOT_SMD:TSOT-23-6, symbol Regulator_Switching:AP63205WU
- C4001: renamed from C42; footprint (none) -> Capacitor_THT:CP_Radial_D6.3mm_P2.50mm; mouser (none) -> 667-EEU-FM1H560
- C4002: renamed from C41; footprint (none) -> Capacitor_THT:CP_Radial_D6.3mm_P2.50mm; mouser (none) -> 667-EEU-FM1H560
- C4003: renamed from C21; footprint (none) -> Capacitor_SMD:C_0805_2012Metric; mouser (none) -> 81-GRM21BR61H106KE3L
- C4004: renamed from C23; footprint (none) -> Capacitor_SMD:C_0805_2012Metric; mouser (none) -> 81-GRM21BR61H106KE3L
- C4005: renamed from C31; footprint (none) -> Capacitor_SMD:C_0805_2012Metric; mouser (none) -> 81-GRM21BR61H106KE3L
- C4006: renamed from C32; footprint (none) -> Capacitor_SMD:C_0805_2012Metric; mouser (none) -> 81-GRM21BR61H106KE3L
- C4007: renamed from C33; footprint (none) -> Capacitor_SMD:C_0805_2012Metric; mouser (none) -> 81-GRM21BR61H106KE3L
- C4008: renamed from C38; footprint (none) -> Capacitor_SMD:C_0805_2012Metric; mouser (none) -> 81-GRM21BR61H106KE3L
- C4009: renamed from C37; footprint (none) -> Capacitor_SMD:C_0805_2012Metric; mouser (none) -> 81-GRM21BR61H106KE3L
- C4010: renamed from C36; footprint (none) -> Capacitor_SMD:C_0805_2012Metric; mouser (none) -> 81-GRM21BR61H106KE3L
- C4011: renamed from C35; footprint (none) -> Capacitor_SMD:C_0805_2012Metric; mouser (none) -> 81-GRM21BR61H106KE3L
- C4012: renamed from C34; footprint (none) -> Capacitor_SMD:C_0805_2012Metric; mouser (none) -> 81-GRM21BR61H106KE3L
- C4013: renamed from C44; footprint (none) -> Capacitor_THT:CP_Radial_D6.3mm_P2.50mm; mouser (none) -> 667-EEU-FM1H560
- C4014: renamed from C43; footprint (none) -> Capacitor_THT:CP_Radial_D6.3mm_P2.50mm; mouser (none) -> 667-EEU-FM1H560
- C4023: renamed from C29; footprint (none) -> Capacitor_SMD:C_0402_1005Metric; mouser (none) -> 81-GRM155R61H105KE5J
- C4024: renamed from C30; footprint (none) -> Capacitor_SMD:C_0402_1005Metric; mouser (none) -> 81-GRM155R61H105KE5J
- C4025: renamed from C28; footprint (none) -> Capacitor_SMD:C_0603_1608Metric; mouser (none) -> 81-GRM188C81C225MA2D
- C4026: renamed from C1; footprint (none) -> Capacitor_SMD:C_0402_1005Metric; mouser (none) -> 81-GRM155R61C102KA1D
- C4027: renamed from C3; footprint (none) -> Capacitor_SMD:C_0805_2012Metric; mouser (none) -> 81-GRM21BR61H106KE3L
- C4028: renamed from C39; footprint (none) -> Capacitor_SMD:C_0402_1005Metric; mouser (none) -> 81-GCM155R71H104KE2D
- C4029: renamed from C40; footprint (none) -> Capacitor_SMD:C_0402_1005Metric; mouser (none) -> 603-CC0402JRX77BB333
- C4030: renamed from C24; footprint (none) -> Capacitor_SMD:C_0402_1005Metric; mouser (none) -> 581-040216C103K
- C4031: renamed from C25; footprint (none) -> Capacitor_SMD:C_0402_1005Metric; mouser (none) -> 81-GRT1555C1H681FA2D
- C4032: renamed from C26; footprint (none) -> Capacitor_SMD:C_0402_1005Metric; mouser (none) -> 81-GRM1555C1H680JA1D
- C4033: renamed from C27; footprint (none) -> Capacitor_SMD:C_0402_1005Metric; mouser (none) -> 80-C0402C101J5GAC
- D4001: renamed from D1; mouser (none) -> 863-BZX84C6V2LT3G
- D4002: renamed from D5; footprint (none) -> Diode_SMD:D_SOD-123; mouser (none) -> 621-SBR0560S1-7-F
- D4003: renamed from D4; footprint (none) -> Diode_SMD:D_SOD-123; mouser (none) -> 621-SBR0560S1-7-F
- D4004: renamed from D2; value LED -> LED-GREEN; footprint (none) -> LED_SMD:LED_0603_1608Metric; mouser (none) -> 710-150060GS75003
- D4005: renamed from D3; value LED -> LED-GREEN; footprint (none) -> LED_SMD:LED_0603_1608Metric; mouser (none) -> 710-150060GS75003
- F4001: renamed from F1; footprint (none) -> Fuse:Fuse_0603_1608Metric; mouser (none) -> 530-C2Q5
- F4002: renamed from F2; value 10A -> 20A; footprint (none) -> Fuse:Fuse_1206_3216Metric; mouser (none) -> 530-C1H20
- J4003: renamed from J1; footprint (none) -> Connector_PinHeader_2.54mm:PinHeader_1x02_P2.54mm_Vertical; ETA (none) -> ETA
- L4003: renamed from L1; footprint (none) -> Inductor_SMD:L_Coilcraft_XAL1010-XXX; mouser (none) -> 994-XAL1010-153MED
- Q4001: renamed from Q8; value Si7960DP -> Si7234DP; mouser (none) -> 781-SI7234DP-T1-GE3
- Q4002: renamed from Q4; value Si7960DP -> Si7234DP; mouser (none) -> 781-SI7234DP-T1-GE3
- Q4003: renamed from Q5; mouser (none) -> 781-SI7461DP-T1-E3
- R4001: renamed from R13; footprint (none) -> Resistor_SMD:R_Shunt_Vishay_WSR2_WSR3_KelvinConnection; mouser (none) -> 71-WSR28L000FEA
- R4003: renamed from R14; footprint (none) -> Resistor_SMD:R_Shunt_Vishay_WSR2_WSR3_KelvinConnection; mouser (none) -> 71-WSR28L000FEA
- R4004: renamed from R21; footprint (none) -> Resistor_SMD:R_0402_1005Metric; mouser (none) -> 71-CRCW0402-215K-E3
- R4005: renamed from R22; footprint (none) -> Resistor_SMD:R_0402_1005Metric; mouser (none) -> 71-CRCW0402-24.9K-E3
- R4006: renamed from R23; footprint (none) -> Resistor_SMD:R_0402_1005Metric; mouser (none) -> 71-CRCW0402100RFKEDC
- R4007: renamed from R2; footprint (none) -> Resistor_SMD:R_0402_1005Metric; mouser (none) -> 71-CRCW0402-105K-E3
- R4008: renamed from R20; footprint (none) -> Resistor_SMD:R_Shunt_Vishay_WSKW0612; mouser (none) -> 71-WSKW06122L000FEA
- R4009: renamed from R1; footprint (none) -> Resistor_SMD:R_0402_1005Metric; mouser (none) -> 71-CRCW0402100RFKEDC
- R4010: renamed from R24; footprint (none) -> Resistor_SMD:R_0402_1005Metric; mouser (none) -> 71-CRCW0402-4.7-E3
- R4011: renamed from R25; footprint (none) -> Resistor_SMD:R_0402_1005Metric; mouser (none) -> 71-CRCW040210K0JNEDC
- R4012: renamed from R26; value 215K -> 215k; footprint (none) -> Resistor_SMD:R_0402_1005Metric; mouser (none) -> 71-CRCW0402-215K-E3
- R4013: renamed from R27; value 24K9 -> 24k9; footprint (none) -> Resistor_SMD:R_0402_1005Metric; mouser (none) -> 71-CRCW0402-24.9K-E3
- R4014: renamed from R17; footprint (none) -> Resistor_SMD:R_0402_1005Metric; mouser (none) -> 71-CRCW0402-100K-E3
- R4015: renamed from R18; footprint (none) -> Resistor_SMD:R_0402_1005Metric; mouser (none) -> 71-CRCW040256K0FKED
- R4016: renamed from R19; footprint (none) -> Resistor_SMD:R_0402_1005Metric; mouser (none) -> 71-CRCW040247K0FKEDC
- R4017: renamed from R15; footprint (none) -> Resistor_SMD:R_0402_1005Metric; mouser (none) -> 71-CRCW04021K00FKEE
- R4018: renamed from R16; footprint (none) -> Resistor_SMD:R_0402_1005Metric; mouser (none) -> 71-CRCW04021K00FKEE
- TH4001: renamed from TH1; mouser (none) -> 504-NRBE104J3380B1J; now not fitted
- U4003: renamed from U5; mouser (none) -> 584-LTC4020EUHFTRPBF
Connections:
- net +3V3: now also C4036.1, C4037.1, L4004.2, TP4012.1, U4004.1 (FB)
- net +5V: now also C4035.1, C4040.1, C4041.1, L4005.2, TP4013.1, U4004.2 (EN), U4004.3 (IN), U4005.1 (FB)
- net BATT_RAW: now also D4006.1 (K)
- net GND: now also Q4002.3 (S), C4035.2, C4036.2, C4037.2, C4039.2, C4040.2, C4041.2, TP4011.1, U4004.4 (GND), U4005.4 (GND)
- net SW1: now also C4023.1
- net SW2: now also D4006.2 (A)
- net TG1: no longer C4023.1
- net at Q4001.3 (S), R4003.4: no longer Q4002.3 (S)
- net at F4002.2: now also TP4010.1
- net CSOUT: now reaches C4033.1, U4003.24 (CSOUT)
- net ITH: now reaches R4015.1, U4003.27 (ITH)
- net VC: now reaches C4032.1, R4016.1, U4003.28 (VC)
- net STAT1_OUT: now reaches D4004.2 (A), R4017.2
- net STAT2_OUT: now reaches D4005.2 (A), R4018.2
- net +BATT renamed +SYSTEM
- net +SYSTEM: now also C4039.1, U4005.2 (EN), U4005.3 (IN)
- new net: J4001.5 (Pin_5), TP4005.1
- new net: J4001.2 (Pin_2), TP4008.1
- new net: J4002.1 (Pin_1), TP4003.1
- new net: C4034.1, L4004.1, U4004.5 (SW)
- new net: C4034.2, U4004.6 (BST)
- new net: J4002.2 (Pin_2), TP4009.1
- new net: J4001.3 (Pin_3), TP4007.1
- new net: J4001.4 (Pin_4), TP4006.1
- new net: J4001.6 (Pin_6), TP4004.1
- new net: C4038.1, L4005.1, U4005.5 (SW)
- new net: C4038.2, U4005.6 (BST)
- no-connect marks 2 -> 4
Other:
- moved on the sheet: C4001, C4002, C4003, C4004, C4005, C4006, C4007, C4008, C4009, C4010, C4011, C4012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

Commit message: User interface fix
Parts:
- J403: renamed from J4003; value Conn_PTC -> Conn_NTC
- renumbered C4034 to C401, C4001 to C402, C4002 to C403, C4003 to C404, C4004 to C405, C4005 to C406, C4006 to C407, C4007 to C408, C4008 to C409, C4009 to C410, C4010 to C411, C4011 to C412, C4012 to C413, C4013 to C414, C4014 to C415, C4035 to C416, C4036 to C417, C4037 to C418, C4038 to C419, C4039 to C420, C4040 to C421, C4041 to C422, C4023 to C423, C4024 to C424, C4025 to C425, C4026 to C426, C4027 to C427, C4030 to C428, C4031 to C429, C4032 to C430, C4033 to C431, C4028 to C432, C4029 to C433, D4006 to D401, D4001 to D402, D4003 to D403, D4002 to D404, D4004 to D405, D4005 to D406, F4001 to F401, F4002 to F402, J4002 to J401, J4001 to J402, L4004 to L401, L4003 to L402, L4005 to L403, Q4001 to Q401, Q4002 to Q402, Q4003 to Q403, R4001 to R401, R4003 to R402, R4006 to R403, R4007 to R404, R4004 to R405, R4012 to R406, R4008 to R407, R4009 to R408, R4010 to R409, R4011 to R410, R4005 to R411, R4013 to R412, R4014 to R413, R4015 to R414, R4016 to R415, R4017 to R416, R4018 to R417, TH4001 to TH401, TP4012 to TP401, TP4013 to TP402, TP4004 to TP403, TP4010 to TP404, TP4009 to TP405, TP4005 to TP406, TP4011 to TP407, TP4003 to TP408, TP4006 to TP409, TP4007 to TP410, TP4008 to TP411, U4004 to U401, U4005 to U402, U4003 to U403
Connections:
- net STAT1 is gone; now on net STAT1_OUT: D405.1 (K), U403.12 (STAT1)
- net STAT2 is gone; now on net STAT2_OUT: D406.1 (K), U403.13 (STAT2)
- net STAT1_OUT: no longer D405.2 (A), R416.2
- net STAT2_OUT: no longer D406.2 (A), R417.2
- new net: D405.2 (A), R416.2
- new net: D406.2 (A), R417.2

Commit message: User interface and Controller done
yes
Parts:
- added R418, R419: 1k, Resistor_SMD:R_0402_1005Metric, symbol Device:R
- added R420, R421: 10k, Resistor_SMD:R_0402_1005Metric, symbol Device:R
- J401: footprint Connector_AMASS:AMASS_XT60IPW-M_1x03_P7.20mm_Horizontal -> Connector_AMASS:AMASS_XT60PW-M_1x02_P7.20mm_Horizontal
- Q401, Q402: value Si7234DP -> Si7252DP; footprint Package_SO:Vishay_PowerPAK_1212-8_Dual -> Package_SO:PowerPAK_SO-8_Dual; mouser 781-SI7234DP-T1-GE3 -> 78-SI7252ADP-T1-GE3
- Q403: footprint Package_SO:Vishay_PowerPAK_1212-8_Single -> Package_SO:PowerPAK_SO-8_Single
- R401, R402: footprint Resistor_SMD:R_Shunt_Vishay_WSR2_WSR3_KelvinConnection -> personal:R_Shunt_Vishay_WSR2_WSR3_KelvinConnection_4pins
Connections:
- net +SYSTEM: now also R420.1
- net BATT_RAW: now also Q402.5 (D), R407.1; no longer Q402.6 (D), R407.4
- net BG1: now also Q401.2 (G); no longer Q401.4 (G)
- net BG2: now also Q402.2 (G); no longer Q402.4 (G)
- net GND: now also Q402.1 (S), R402.4, R418.1, R419.1; no longer Q402.3 (S), R402.1
- net SENSBOT: now also R402.2; no longer R402.3
- net SENSGND: now also R402.3; no longer R402.2
- net SENSTOP: now also R401.3; no longer R401.2
- net SENSVin: now also R401.2; no longer R401.3
- net SW1: now also Q401.3 (S), Q401.6 (D); no longer Q401.1 (S), Q401.5 (D)
- net SW2: now also Q402.3 (S), Q402.6 (D); no longer Q402.1 (S), Q402.5 (D)
- net TG1: now also Q401.4 (G); no longer Q401.2 (G)
- net TG2: now also Q402.4 (G); no longer Q402.2 (G)
- net VBUS: now also R401.1, R421.1; no longer R401.4
- net at C426.1, R408.2: now also R407.3; no longer R407.2
- net at R403.2: now also R407.2; no longer R407.3
- net at Q403.5 (D): now also R407.4; no longer R407.1
- new net: Q401.5 (D), R401.4
- new net: Q401.1 (S), R402.1
- new net BATTERY_MONITOR: R419.2, R420.2
- new net VBUS_MONITOR: R418.2, R421.2
Other:
- moved on the sheet: D401, Q401A, Q401B, Q402A, Q402B, R401, R402, R407
