File: Hardware/Controller/Controller.kicad_sch (KiCad schematic)
At the start: 0 parts

Commit message: Controller fixades
Other:
- added sheet CAN_bus (CAN_bus.kicad_sch)
- sheet Battery ports: added 5V_EN, STAT1, STAT2; removed none
- sheet Microcontroller ports: added GPIO0, GPIO1, GPIO10, GPIO11, GPIO12, GPIO13, GPIO14, GPIO15, GPIO16, GPIO17, GPIO18, GPIO19, GPIO2, GPIO20, GPIO21, GPIO22, GPIO23, GPIO24, GPIO25, GPIO26_ADC0, GPIO27_ADC1, GPIO28_ADC2, GPIO29_ADC3, GPIO3, GPIO4, GPIO5, GPIO6, GPIO7, GPIO8, GPIO9, USB_D+, USB_D-; removed none
- sheet USBC ports: added CFG2, CFG3, PG, POWEROUT, USB_D+, USB_D-, ~{CFG1}; removed none
- company: (none) -> Chalmers EENX16-VT24-27

Commit message: User interface and Controller done
yes
Parts:
- added H101, H102, H103, H104: MountingHole, MountingHole:MountingHole_3.2mm_M3, symbol Mechanical:MountingHole
Other:
- sheet Battery ports: added BATTERY_MONITOR, STAT1_OUT, STAT2_OUT, VBUS_MONITOR; removed 5V_EN, STAT1, STAT2
- sheet USBC ports: added none; removed POWEROUT

Commit message: final fixes (hopefully) (GONE WRONG?!) (real)
Other:
- title: (none) -> Illumination system controller - overview

Commit message: Add software files
Other:
- sheet USBC ports: added none; removed CFG2, CFG3, ~{CFG1}
Changed lines of the file:
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@@
-	(wire
-		(pts
-			(xy 66.04 48.26) (xy 64.77 48.26)
-		)
-		(stroke
-			(width 0)
-			(type default)
-		)
-	)
 	(wire
 		(pts
@@
 	(wire
 		(pts
-			(xy 66.04 50.8) (xy 64.77 50.8)
-		)
-		(stroke
-			(width 0)
-			(type default)
-		)
-	)
-	(wire
-		(pts
 			(xy 105.41 72.39) (xy 106.68 72.39)
 		)
@@
 	(wire
 		(pts
-			(xy 105.41 44.45) (xy 106.68 44.45)
-		)
-		(stroke
-			(width 0)
-			(type default)
-		)
-	)
-	(wire
-		(pts
 			(xy 105.41 26.67) (xy 106.68 26.67)
 		)
@@
 	(wire
 		(pts
-			(xy 105.41 41.91) (xy 106.68 41.91)
-		)
-		(stroke
-			(width 0)
-			(type default)
-		)
-	)
-	(wire
-		(pts
 			(xy 64.77 91.44) (xy 66.04 91.44)
 		)
@@
 	(wire
 		(pts
-			(xy 66.04 53.34) (xy 64.77 53.34)
-		)
-		(stroke
-			(width 0)
-			(type default)
-		)
-	)
-	(wire
-		(pts
 			(xy 66.04 118.11) (xy 64.77 118.11)
 		)
@@
 		(pts
 			(xy 64.77 93.98) (xy 66.04 93.98)
-		)
-		(stroke
-			(width 0)
-			(type default)
-		)
-	)
-	(wire
-		(pts
-			(xy 105.41 39.37) (xy 106.68 39.37)
 		)
 		(stroke
@@
 		)
 	)
-	(label "~{CFG1}"
-		(at 105.41 44.45 180)
-		(fields_autoplaced yes)
-		(effects
-			(font
-				(size 1.27 1.27)
-			)
-			(justify right bottom)
-		)
-	)
 	(label "USB_D-"
 		(at 105.41 26.67 180)
@@
 		)
 	)
-	(label "~{CFG1}"
-		(at 66.04 53.34 0)
-		(fields_autoplaced yes)
-		(effects
-			(font
-				(size 1.27 1.27)
-			)
-			(justify left bottom)
-		)
-	)
 	(label "~{CS}"
 		(at 105.41 102.87 180)
@@
 		)
 	)
-	(label "CFG2"
-		(at 66.04 50.8 0)
-		(fields_autoplaced yes)
-		(effects
-			(font
-				(size 1.27 1.27)
-			)
-			(justify left bottom)
-		)
-	)
 	(label "VBUS_MONITOR"
 		(at 66.04 115.57 0)
@@
 		)
 	)
-	(label "CFG2"
-		(at 105.41 41.91 180)
-		(fields_autoplaced yes)
-		(effects
-			(font
-				(size 1.27 1.27)
-			)
-			(justify right bottom)
-		)
-	)
 	(label "STAT2_OUT"
 		(at 66.04 76.2 0)
@@
 		)
 	)
-	(label "CFG3"
-		(at 66.04 48.26 0)
-		(fields_autoplaced yes)
-		(effects
-			(font
-				(size 1.27 1.27)
-			)
-			(justify left bottom)
-		)
-	)
 	(label "PG"
 		(at 105.41 34.29 180)
@@
 	(label "~{INT}"
 		(at 105.41 105.41 180)
-		(fields_autoplaced yes)
-		(effects
-			(font
-				(size 1.27 1.27)
-			)
-			(justify right bottom)
-		)
-	)
-	(label "CFG3"
-		(at 105.41 39.37 180)
 		(fields_autoplaced yes)
 		(effects
@@
 			(effects
 				(font
-					(size 1.27 1.27)
-				)
-				(justify left)
-			)
-		)
-		(pin "CFG3" input
-			(at 106.68 39.37 180)
-			(effects
-				(font
-					(size 1.27 1.27)
-				)
-				(justify left)
-			)
-		)
-		(pin "CFG2" input
-			(at 106.68 41.91 180)
-			(effects
-				(font
-					(size 1.27 1.27)
-				)
-				(justify left)
-			)
-		)
-		(pin "~{CFG1}" input
-			(at 106.68 44.45 180)
-			(effects
-				(font
