File: Hardware/Controller/USBC.kicad_sch (KiCad schematic)
At the start: 12 parts, among them J4 USB_C_Receptacle_USB2.0_16P, Q1 Q_NMOS_GSD, U4 CH224K

Commit message: Controller fixades
Connections:
- net POWEROUT renamed VBUS
Other:
- company: (none) -> Chalmers EENX16-VT24-27
- title: (none) -> USB-C + Power Delivery
Changed lines of the file:
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@@
 	(generator_version "8.0")
 	(paper "A4")
+	(title_block
+		(title "USB-C + Power Delivery")
+		(date "2024-03-01")
+		(rev "A01")
+		(company "Chalmers EENX16-VT24-27")
+	)
 	(junction
 		(at 133.35 60.96)
@@
 	(wire
 		(pts
-			(xy 176.53 30.48) (xy 189.23 30.48)
+			(xy 176.53 30.48) (xy 186.69 30.48)
 		)
 		(stroke
@@
 		(shape input)
 		(at 162.56 71.12 0)
-		(fields_autoplaced yes)
-		(effects
-			(font
-				(size 1.27 1.27)
-			)
-			(justify left)
-		)
-	)
-	(hierarchical_label "POWEROUT"
-		(shape output)
-		(at 189.23 30.48 0)
 		(fields_autoplaced yes)
 		(effects
@@
 					(unit 1)
 				)
+			)
+		)
+	)
+	(symbol
+		(lib_id "power:VBUS")
+		(at 186.69 30.48 0)
+		(unit 1)
+		(exclude_from_sim no)
+		(in_bom yes)
+		(on_board yes)
+		(dnp no)
+		(fields_autoplaced yes)
+		(property "Reference" "#PWR068"
+			(at 186.69 34.29 0)
+			(effects
+				(font
+					(size 1.27 1.27)
+				)
+				(hide yes)
+			)
+		)
+		(property "Value" "VBUS"
+			(at 186.69 25.4 0)
+			(effects
+				(font
+					(size 1.27 1.27)
+				)
+			)
+		)
+		(property "Footprint" ""
+			(at 186.69 30.48 0)
+			(effects
+				(font
+					(size 1.27 1.27)
+				)
+				(hide yes)
+			)
+		)
+		(property "Datasheet" ""
+			(at 186.69 30.48 0)
+			(effects
+				(font
+					(size 1.27 1.27)
+				)
+				(hide yes)
+			)
+		)
+		(property "Description" "Power symbol creates a global label with name \"VBUS\""
+			(at 186.69 30.48 0)
+			(effects
+				(font
+					(size 1.27 1.27)
+				)
+				(hide yes)
+			)
+		)
+		(pin "1"
+		)
+		(instances
+			(project "Controller"
+				(path "/43ebced7-8538-4711-b1b5-1811dcfcbefa/65228501-681e-424e-8fc1-d56cc57cdfa3"
+					(reference "#PWR068")
+					(unit 1)
+				)

Commit message: La in allt
Myyycket saker
Parts:
- removed J4: USB_C_Receptacle_USB2.0_16P, symbol Connector:USB_C_Receptacle_USB2.0_16P
- added J3001: USB_C_Receptacle_USB2.0_16P, Connector_USB:USB_C_Receptacle_GCT_USB4105-xx-A_16P_TopMnt_Horizontal, symbol Connector:USB_C_Receptacle_USB2.0_16P
- C3001: renamed from C18; mouser 81-GRM21BR61H106KE3L -> 81-GRM21BR61H106KE3L
- C3002: renamed from C19; mouser 81-GRM21BR61H106KE3L -> 81-GRM21BR61H106KE3L
- C3003: renamed from C20; mouser 81-GRM21BR61H106KE3L -> 81-GRM21BR61H106KE3L
- C3004: renamed from C22; mouser 81-GRM155R61H105KE5J -> 81-GRM155R61H105KE5J
- Q3001: renamed from Q1; ETA (none) -> ETA
- R3001: renamed from R8; mouser 71-CRCW04021K00FKEE -> 71-CRCW04021K00FKEE
- R3002: renamed from R9; mouser 71-CRCW040210K0JNEDC -> 71-CRCW040210K0JNEDC
- R3003: renamed from R10; mouser 71-CRCW040210K0JNEDC -> 71-CRCW040210K0JNEDC
- R3004: renamed from R11; mouser 71-CRCW040210K0JNEDC -> 71-CRCW040210K0JNEDC
- R3005: renamed from R12; mouser 71-CRCW040210K0JNEDC -> 71-CRCW040210K0JNEDC
- U3001: renamed from U4; ETA (none) -> ETA
Connections:
- net CC1: now also J3001.A5 (CC1)
- net CC2: now also J3001.B5 (CC2)
- net GND: now also J3001.A1 (GND), J3001.A12 (GND), J3001.B1 (GND), J3001.B12 (GND)
- net USB_D+: now also J3001.A6 (D+), J3001.B6 (D+)
- net USB_D-: now also J3001.A7 (D-), J3001.B7 (D-)
- net VBUS: now also J3001.A4 (VBUS), J3001.A9 (VBUS), J3001.B4 (VBUS), J3001.B9 (VBUS)
Other:
- moved on the sheet: C3002, C3003, C3004

Commit message: User interface fix
Parts:
- renumbered C3001 to C301, C3002 to C302, C3003 to C303, C3004 to C304, J3001 to J301, Q3001 to Q301, R3001 to R301, R3002 to R302, R3003 to R303, R3004 to R304, R3005 to R305, U3001 to U301
Changed lines of the file:
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@@
 		(on_board yes)
 		(dnp no)
-		(property "Reference" "#PWR03003"
+		(property "Reference" "#PWR0303"
 			(at 133.35 53.34 0)
 			(effects
@@
 			(project "Controller"
 				(path "/43ebced7-8538-4711-b1b5-1811dcfcbefa/65228501-681e-424e-8fc1-d56cc57cdfa3"
-					(reference "#PWR03003")
+					(reference "#PWR0303")
 					(unit 1)
 				)
@@
 		(on_board yes)
 		(dnp no)
-		(property "Reference" "Q3001"
+		(property "Reference" "Q301"
 			(at 146.05 77.47 0)
 			(effects
@@
 			(project "Controller"
 				(path "/43ebced7-8538-4711-b1b5-1811dcfcbefa/65228501-681e-424e-8fc1-d56cc57cdfa3"
-					(reference "Q3001")
+					(reference "Q301")
 					(unit 1)
 				)
@@
 		(dnp no)
 		(fields_autoplaced yes)
-		(property "Reference" "J3001"
+		(property "Reference" "J301"
 			(at 44.45 24.13 0)
 			(effects
@@
 			(project "Controller"
 				(path "/43ebced7-8538-4711-b1b5-1811dcfcbefa/65228501-681e-424e-8fc1-d56cc57cdfa3"
-					(reference "J3001")
+					(reference "J301")
 					(unit 1)
 				)
@@
 		(dnp no)
 		(fields_autoplaced yes)
-		(property "Reference" "#PWR03001"
+		(property "Reference" "#PWR0301"
 			(at 181.61 34.29 0)
 			(effects
@@
 			(project "Controller"
 				(path "/43ebced7-8538-4711-b1b5-1811dcfcbefa/65228501-681e-424e-8fc1-d56cc57cdfa3"
-					(reference "#PWR03001")
+					(reference "#PWR0301")
 					(unit 1)
 				)
@@
 		(dnp no)
 		(fields_autoplaced yes)
-		(property "Reference" "U3001"
+		(property "Reference" "U301"
 			(at 121.5741 81.28 0)
 			(effects
@@
 			(project "Controller"
 				(path "/43ebced7-8538-4711-b1b5-1811dcfcbefa/65228501-681e-424e-8fc1-d56cc57cdfa3"
-					(reference "U3001")
+					(reference "U301")
 					(unit 1)
 				)
@@
 		(on_board yes)
 		(dnp no)
-		(property "Reference" "R3002"
+		(property "Reference" "R302"
 			(at 124.46 37.846 0)
 			(effects
@@
 			(project "Controller"
 				(path "/43ebced7-8538-4711-b1b5-1811dcfcbefa/65228501-681e-424e-8fc1-d56cc57cdfa3"
-					(reference "R3002")
+					(reference "R302")
 					(unit 1)
 				)
@@
 		(on_board yes)
 		(dnp no)
-		(property "Reference" "R3005"
+		(property "Reference" "R305"
 			(at 159.766 82.296 0)
 			(effects
@@
 			(project "Controller"
 				(path "/43ebced7-8538-4711-b1b5-1811dcfcbefa/65228501-681e-424e-8fc1-d56cc57cdfa3"
-					(reference "R3005")
+					(reference "R305")
 					(unit 1)
 				)
@@
 		(on_board yes)
 		(dnp no)
-		(property "Reference" "R3003"
+		(property "Reference" "R303"
 			(at 134.62 52.07 0)
 			(effects
@@
 			(project "Controller"
 				(path "/43ebced7-8538-4711-b1b5-1811dcfcbefa/65228501-681e-424e-8fc1-d56cc57cdfa3"
-					(reference "R3003")
+					(reference "R303")
 					(unit 1)
 				)
@@
 		(on_board yes)
 		(dnp no)
-		(property "Reference" "R3004"
+		(property "Reference" "R304"
 			(at 151.13 63.5 0)
 			(effects
@@
 			(project "Controller"
 				(path "/43ebced7-8538-4711-b1b5-1811dcfcbefa/65228501-681e-424e-8fc1-d56cc57cdfa3"
-					(reference "R3004")
+					(reference "R304")
 					(unit 1)
 				)
@@
 		(on_board yes)
 		(dnp no)
-		(property "Reference" "C3003"
+		(property "Reference" "C303"
 			(at 181.61 31.75 0)
 			(effects
@@
 			(project "Controller"
 				(path "/43ebced7-8538-4711-b1b5-1811dcfcbefa/65228501-681e-424e-8fc1-d56cc57cdfa3"
-					(reference "C3003")
+					(reference "C303")
 					(unit 1)
 				)
@@
 		(dnp no)
 		(fields_autoplaced yes)
-		(property "Reference" "#PWR03004"
+		(property "Reference" "#PWR0304"
 			(at 99.06 59.69 0)
 			(effects
@@
 			(project "Controller"
 				(path "/43ebced7-8538-4711-b1b5-1811dcfcbefa/65228501-681e-424e-8fc1-d56cc57cdfa3"
-					(reference "#PWR03004")
+					(reference "#PWR0304")
 					(unit 1)
 				)
@@
 		(on_board yes)
 		(dnp no)
-		(property "Reference" "R3001"
+		(property "Reference" "R301"
 			(at 114.3 37.592 0)
 			(effects
@@
 			(project "Controller"
 				(path "/43ebced7-8538-4711-b1b5-1811dcfcbefa/65228501-681e-424e-8fc1-d56cc57cdfa3"
-					(reference "R3001")
+					(reference "R301")
 					(unit 1)
 				)
@@
 		(dnp no)
 		(fields_autoplaced yes)
-		(property "Reference" "#PWR03005"
+		(property "Reference" "#PWR0305"
 			(at 44.45 74.93 0)
 			(effects
@@
 			(project "Controller"
 				(path "/43ebced7-8538-4711-b1b5-1811dcfcbefa/65228501-681e-424e-8fc1-d56cc57cdfa3"
-					(reference "#PWR03005")
+					(reference "#PWR0305")
 					(unit 1)
 				)
@@
 		(on_board yes)
 		(dnp no)
-		(property "Reference" "C3004"
+		(property "Reference" "C304"
 			(at 99.06 46.99 0)
 			(effects
@@
 			(project "Controller"
 				(path "/43ebced7-8538-4711-b1b5-1811dcfcbefa/65228501-681e-424e-8fc1-d56cc57cdfa3"
-					(reference "C3004")
+					(reference "C304")
 					(unit 1)
 				)
@@
 		(on_board yes)
 		(dnp no)
-		(property "Reference" "C3001"
+		(property "Reference" "C301"
 			(at 166.37 31.75 0)
 			(effects
@@
 			(project "Controller"
 				(path "/43ebced7-8538-4711-b1b5-1811dcfcbefa/65228501-681e-424e-8fc1-d56cc57cdfa3"
-					(reference "C3001")
+					(reference "C301")
 					(unit 1)
 				)
@@
 		(on_board yes)
 		(dnp no)
-		(property "Reference" "C3002"
+		(property "Reference" "C302"
 			(at 173.99 31.75 0)
 			(effects
@@
 			(project "Controller"
 				(path "/43ebced7-8538-4711-b1b5-1811dcfcbefa/65228501-681e-424e-8fc1-d56cc57cdfa3"
-					(reference "C3002")
+					(reference "C302")
 					(unit 1)
 				)
@@
 		(dnp no)
 		(fields_autoplaced yes)
-		(property "Reference" "#PWR03007"
+		(property "Reference" "#PWR0307"
 			(at 149.86 95.25 0)
 			(effects
@@
 			(project "Controller"
 				(path "/43ebced7-8538-4711-b1b5-1811dcfcbefa/65228501-681e-424e-8fc1-d56cc57cdfa3"
-					(reference "#PWR03007")
+					(reference "#PWR0307")
 					(unit 1)
 				)
@@
 		(dnp no)
 		(fields_autoplaced yes)
-		(property "Reference" "#PWR03006"
+		(property "Reference" "#PWR0306"
 			(at 119.38 87.63 0)
 			(effects
@@
 			(project "Controller"
 				(path "/43ebced7-8538-4711-b1b5-1811dcfcbefa/65228501-681e-424e-8fc1-d56cc57cdfa3"
-					(reference "#PWR03006")
+					(reference "#PWR0306")
 					(unit 1)
 				)
@@
 		(dnp no)
 		(fields_autoplaced yes)
-		(property "Reference" "#PWR03002"
+		(property "Reference" "#PWR0302"
 			(at 181.61 44.45 0)
 			(effects
@@
 			(project "Controller"
 				(path "/43ebced7-8538-4711-b1b5-1811dcfcbefa/65228501-681e-424e-8fc1-d56cc57cdfa3"
-					(reference "#PWR03002")
-					(unit 1)
-				)
+					(reference "#PWR0302")
+					(unit 1)
+				)

Commit message: Add software files
Parts:
- removed Q301: Q_NMOS_GSD, Package_TO_SOT_SMD:SOT-23-3, symbol Device:Q_NMOS_GSD
- added R306: 10k, Resistor_SMD:R_0402_1005Metric, symbol Device:R
Connections:
- net CFG2 is gone; now on an unnamed net: U301.2 (CFG2)
- net ~{CFG1} is gone; now on an unnamed net: R305.1
- net GND: now also R306.2
- net at R304.2: no longer U301.9 (CFG1)
- net CFG3: no longer names the net of U301.3 (CFG3)
- new net: R306.1, U301.9 (CFG1)
Other:
- moved on the sheet: R304
