File: Hardware/UserInterface/CAN_Bus+power.kicad_sch (KiCad schematic)
At the start: 33 parts, among them J3 RJ10, J4 RJ10, U4 MCP2515-xST, U5 MCP2551-I-SN, U6 AP63203WU, U7 AP63205WU, Y2 8M

Commit message: User interface fix
Parts:
- removed C18, C19: C, symbol Device:C
- removed C20, C21: 100n, symbol Device:C
- removed C22, C23, C24, C25, C28, C29, C30, C31: 10u, symbol Device:C
- removed C26, C27: 100n, symbol Device:C_Small
- removed F1: 4A, symbol Device:Fuse
- removed J3, J4: RJ10, Connector_RJ:RJ9_Evercom_5301-440xxx_Horizontal, symbol Connector:RJ10
- removed JP2: Jumper_termination, symbol Jumper:Jumper_2_Open
- removed L1, L2: 4u7, symbol Device:L
- removed R10, R11, R8: 10k, symbol Device:R
- removed R12: 120, symbol Device:R_Small
- removed R9: 5k, symbol Device:R
- removed TP1: TPVin, symbol Connector:TestPoint
- removed TP2: TP3V3, symbol Connector:TestPoint
- removed TP3: TP5V, symbol Connector:TestPoint
- removed U4: MCP2515-xST, Package_SO:TSSOP-20_4.4x6.5mm_P0.65mm, symbol Interface_CAN_LIN:MCP2515-xST
- removed U5: MCP2551-I-SN, Package_SO:SOIC-8_3.9x4.9mm_P1.27mm, symbol Interface_CAN_LIN:MCP2551-I-SN
- removed U6: AP63203WU, Package_TO_SOT_SMD:TSOT-23-6, symbol Regulator_Switching:AP63203WU
- removed U7: AP63205WU, Package_TO_SOT_SMD:TSOT-23-6, symbol Regulator_Switching:AP63205WU
- removed Y2: 8M, symbol Device:Crystal_GND23
- added C301, C302, C308, C312: 10u, Capacitor_SMD:C_1206_3216Metric, symbol Device:C
- added C303, C304: 100n, Capacitor_SMD:C_0402_1005Metric, symbol Device:C
- added C305, C306: 10p, Capacitor_SMD:C_0402_1005Metric, symbol Device:C
- added C307, C311: 100n, Capacitor_SMD:C_0402_1005Metric, symbol Device:C_Small
- added C309, C310, C313, C314: 22u, Capacitor_SMD:C_0805_2012Metric, symbol Device:C
- added F301: 4A, Fuse:Fuse_0603_1608Metric, symbol Device:Fuse
- added J301, J302: RJ9, Connector_RJ:RJ9_Evercom_5301-440xxx_Horizontal, symbol Connector:RJ10
- added JP301: Jumper_termination, Connector_PinHeader_2.54mm:PinHeader_1x02_P2.54mm_Vertical, symbol Jumper:Jumper_2_Open
- added L301, L302: 4u7, Inductor_SMD:L_1210_3225Metric, symbol Device:L
- added R301: 120, Resistor_SMD:R_0402_1005Metric, symbol Device:R_Small
- added R302: 5k1, Resistor_SMD:R_0402_1005Metric, symbol Device:R
- added R303, R304, R305: 10k, Resistor_SMD:R_0402_1005Metric, symbol Device:R
- added TP301: TPVin, TestPoint:TestPoint_Pad_D2.0mm, symbol Connector:TestPoint
- added TP302: TP3V3, TestPoint:TestPoint_Pad_D2.0mm, symbol Connector:TestPoint
- added TP303: TP5V, TestPoint:TestPoint_Pad_D2.0mm, symbol Connector:TestPoint
- added U301: MCP2551-I-SN, Package_SO:SOIC-8_3.9x4.9mm_P1.27mm, symbol Interface_CAN_LIN:MCP2551-I-SN
- added U302: MCP2515-xST, Package_SO:TSSOP-20_4.4x6.5mm_P0.65mm, symbol Interface_CAN_LIN:MCP2515-xST
- added U303: AP63203WU, Package_TO_SOT_SMD:TSOT-23-6, symbol Regulator_Switching:AP63203WU
- added U304: AP63205WU, Package_TO_SOT_SMD:TSOT-23-6, symbol Regulator_Switching:AP63205WU
- added Y301: 8M, Crystal:Crystal_SMD_Abracon_ABM3B-4Pin_5.0x3.2mm, symbol Device:Crystal_GND23
Connections:
- net +3V3: now also C303.1, C309.1, C310.1, L301.2, R305.1, TP302.1, U302.20 (VDD), U303.1 (FB)
- net +5V: now also C304.1, C308.1, C313.1, C314.1, L302.2, TP303.1, U301.3 (VDD), U303.2 (EN), U303.3 (IN), U304.1 (FB)
- net +SYSTEM: now also C301.1, C302.1, C312.1, F301.2, TP301.1, U304.2 (EN), U304.3 (IN)
- net CANH: now also J301.2, J302.2, JP301.1 (A), U301.7 (CANH)
- net CANL: now also J301.3, J302.3, R301.2, U301.6 (CANL)
- net GND: now also C301.2, C302.2, C303.2, C304.2, C305.1, C306.1, C308.2, C309.2, C310.2, C312.2, C313.2, C314.2, J301.1, J302.1, R303.2, R304.2, U301.2 (VSS), U302.10 (VSS), U303.4 (GND), U304.4 (GND), Y301.2, Y301.3
- net MISO: now also U302.17 (SO)
- net MOSI: now also U302.16 (SI)
- net SCK: now also U302.14 (SCK)
- net ~{CS}: now also U302.18 (~{CS})
- net ~{INT}: now also U302.13 (~{INT})
- new net: JP301.2 (B), R301.1
- new net: C311.1, L302.1, U304.5 (SW)
- new net: R302.1, U301.4 (RXD)
- new net: R302.2, R303.1, U302.2 (RXCAN)
- new net: F301.1, J301.4, J302.4
- new net: C307.1, L301.1, U303.5 (SW)
- new net: C307.2, U303.6 (BST)
- new net: U301.1 (TXD), U302.1 (TXCAN)
- new net: R305.2, U302.19 (~{RESET})
- new net: C305.2, U302.8 (OSC2), Y301.4
- new net: C306.2, U302.9 (OSC1), Y301.1
- new net: R304.1, U301.8 (Rs)
- new net: C311.2, U304.6 (BST)
Other:
- note removed: "22u kanske?"

Commit message: User interface and Controller done
yes
Parts:
- C301, C302, C308, C312: footprint Capacitor_SMD:C_1206_3216Metric -> Capacitor_SMD:C_0805_2012Metric; mouser 581-1206DD106MAT2A -> 81-GRM21BR61H106KE3L
- Y301: symbol Device:Crystal_GND23 -> Device:Crystal_GND24
Connections:
- net GND: now also Y301.4; no longer Y301.3
- net at C305.2, U302.8 (OSC2): now also Y301.3; no longer Y301.4
Changed lines of the file:
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@@
 			)
 		)
-		(property "Footprint" "Capacitor_SMD:C_1206_3216Metric"
+		(property "Footprint" "Capacitor_SMD:C_0805_2012Metric"
 			(at 230.8352 41.91 0)
 			(effects
@@
 			)
 		)
-		(property "Datasheet" "https://www.mouser.se/datasheet/2/40/cx5r_KGM-3223198.pdf"
+		(property "Datasheet" ""
 			(at 229.87 38.1 0)
 			(effects
@@
 			)
 		)
-		(property "mouser" "581-1206DD106MAT2A"
+		(property "mouser" "81-GRM21BR61H106KE3L"
 			(at 229.87 38.1 0)
 			(effects
@@
 			)
 		)
-		(property "Footprint" "Capacitor_SMD:C_1206_3216Metric"
+		(property "Footprint" "Capacitor_SMD:C_0805_2012Metric"
 			(at 26.3652 184.15 0)
 			(effects
@@
 			)
 		)
-		(property "Datasheet" "https://www.mouser.se/datasheet/2/40/cx5r_KGM-3223198.pdf"
+		(property "Datasheet" ""
 			(at 25.4 180.34 0)
 			(effects
@@
 			)
 		)
-		(property "mouser" "581-1206DD106MAT2A"
+		(property "mouser" "81-GRM21BR61H106KE3L"
 			(at 25.4 180.34 0)
 			(effects
@@
 	)
 	(symbol
-		(lib_id "Device:Crystal_GND23")
+		(lib_id "Device:Crystal_GND24")
 		(at 52.07 93.98 90)
 		(unit 1)
@@
 			)
 		)
-		(property "Datasheet" "https://www.mouser.se/datasheet/2/3/abm3b-1774998.pdf"
+		(property "Datasheet" "~"
 			(at 52.07 93.98 0)
 			(effects
@@
 			)
 		)
-		(property "Description" ""
+		(property "Description" "Four pin crystal, GND on pins 2 and 4"
 			(at 52.07 93.98 0)
 			(effects
@@
 			)
 		)
-		(property "Footprint" "Capacitor_SMD:C_1206_3216Metric"
+		(property "Footprint" "Capacitor_SMD:C_0805_2012Metric"
 			(at 26.3652 144.78 0)
 			(effects
@@
 			)
 		)
-		(property "Datasheet" "https://www.mouser.se/datasheet/2/40/cx5r_KGM-3223198.pdf"
+		(property "Datasheet" ""
 			(at 25.4 140.97 0)
 			(effects
@@
 			)
 		)
-		(property "mouser" "581-1206DD106MAT2A"
+		(property "mouser" "81-GRM21BR61H106KE3L"
 			(at 25.4 140.97 0)
 			(effects
@@
 			)
 		)
-		(property "Footprint" "Capacitor_SMD:C_1206_3216Metric"
+		(property "Footprint" "Capacitor_SMD:C_0805_2012Metric"
 			(at 240.9952 41.91 0)
 			(effects
@@
 			)
 		)
-		(property "Datasheet" "https://www.mouser.se/datasheet/2/40/cx5r_KGM-3223198.pdf"
+		(property "Datasheet" ""
 			(at 240.03 38.1 0)
 			(effects
@@
 			)
 		)
-		(property "mouser" "581-1206DD106MAT2A"
+		(property "mouser" "81-GRM21BR61H106KE3L"
 			(at 240.03 38.1 0)
 			(effects

Commit message: final fixes (hopefully) (GONE WRONG?!) (real)
Other:
- company: (none) -> Chalmers EENX16-VT24-27
- title: (none) -> CAN Bus controller + interface, and power management
Changed lines of the file:
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@@
 	(generator_version "8.0")
 	(paper "A4")
+	(title_block
+		(title "CAN Bus controller + interface, and power management")
+		(date "2024-03-26")
+		(rev "A01")
+		(company "Chalmers EENX16-VT24-27")
+	)
 	(junction
 		(at 229.87 34.29)
