File: Hardware/UserInterface/UserInterface.kicad_sch (KiCad schematic)
At the start: 11 parts, among them J5 conn_OLED, SW3 SW_Push, SW4 SW_Push, SW5 SW_Push, SW6 SW_Push, SW7 SW_Push

Commit message: User interface fix
Parts:
- removed C32, C33, C34, C35, C36: 100n, symbol Device:C
- removed SW3, SW4, SW5, SW6, SW7: SW_Push, symbol Switch:SW_Push
- added C101, C102: 100n, Capacitor_SMD:C_0402_1005Metric, symbol Device:C
- added J101: conn_turnSignal, Connector_PinHeader_2.54mm:PinHeader_1x03_P2.54mm_Vertical, symbol Connector_Generic:Conn_01x03
- added J103: conn_joystick, Connector_PinHeader_2.54mm:PinHeader_1x05_P2.54mm_Vertical, symbol Connector_Generic:Conn_01x05
- J102: renamed from J5; footprint (none) -> Connector_PinHeader_2.54mm:PinHeader_1x04_P2.54mm_Vertical; ETA (none) -> CASE
Connections:
- net GND: now also J102.4 (Pin_4), C101.2, C102.1, J101.2 (Pin_2), J103.5 (Pin_5)
- net SDA: now reaches J102.1 (Pin_1)
- net SCL: now reaches J102.2 (Pin_2)
- net +3V3: now reaches J102.3 (Pin_3)
- net +3V3: now also J103.4 (Pin_4)
- new net BTN: J103.1 (Pin_1)
- new net BTN_LEFT: C102.2, J101.3 (Pin_3)
- new net BTN_RIGHT: C101.1, J101.1 (Pin_1)
- new net VR_x: J103.3 (Pin_3)
- new net VR_y: J103.2 (Pin_2)
Other:
- moved on the sheet: J102

Commit message: User interface and Controller done
yes
Connections:
- no-connect marks 0 -> 1
Other:
- sheet CAN_Bus+power ports: added MISO, MOSI, SCK, ~{CS}, ~{INT}; removed none
- sheet Microcontroller ports: added GPIO0, GPIO1, GPIO10, GPIO11, GPIO12, GPIO13, GPIO14, GPIO15, GPIO16, GPIO17, GPIO18, GPIO19, GPIO2, GPIO20, GPIO21, GPIO22, GPIO23, GPIO24, GPIO25, GPIO26_ADC0, GPIO27_ADC1, GPIO28_ADC2, GPIO29_ADC3, GPIO3, GPIO4, GPIO5, GPIO6, GPIO7, GPIO8, GPIO9; removed none
- moved on the sheet: C101, C102, J101, J102, J103

Commit message: final fixes (hopefully) (GONE WRONG?!) (real)
Other:
- company: (none) -> Chalmers EENX16-VT24-27
- title: (none) -> Illumination system user interface - overview
- moved on the sheet: C101, C102, J101, J102, J103
