File: Hardware/UserInterface/UserInterface.kicad_pcb (KiCad board)
At the start: 2 copper layers, 68 parts, among them J1001 conn_joystick, J1002 conn_turnSignal, J2001 USB_C_Receptacle_USB2.0_16P, J2002 TagConnect_SWD, J3001 RJ9, J3002 RJ9, J5 conn_OLED, SW2001 SW_Push, SW2002 SW_Push, U2001 W25Q64JVXGIQ, U2002 RP2040, U3001 AP63203WU, U3002 AP63205WU, U3003 MCP2551-I-SN, U3004 MCP2515-xST, Y2001 12M, Y3001 8M

Commit message: User interface and Controller done
yes
Parts:
- C301: renamed from C3009; footprint Capacitor_SMD:C_1206_3216Metric -> Capacitor_SMD:C_0805_2012Metric
- C302: renamed from C3010; footprint Capacitor_SMD:C_1206_3216Metric -> Capacitor_SMD:C_0805_2012Metric
- C308: renamed from C3002; footprint Capacitor_SMD:C_1206_3216Metric -> Capacitor_SMD:C_0805_2012Metric
- C312: renamed from C3006; footprint Capacitor_SMD:C_1206_3216Metric -> Capacitor_SMD:C_0805_2012Metric
- moved U201 50.9 mm to (132.6, 40.2)
- moved TP301 48.7 mm to (111.5, 53.8)
- moved F301 46.2 mm to (111.5, 51.5)
- moved D201 45.8 mm to (133.5, 34.5)
- moved JP301 44.6 mm to (118.7, 31.5)
- moved J201 44.1 mm to (148.6, 49.5)
- moved U301 43.9 mm to (114.0, 33.4), turned to 90 degrees
- moved C302 42.4 mm to (111.9, 49.0), turned to 90 degrees
- moved C312 42.0 mm to (114.8, 51.8)
- moved R206 41.8 mm to (143.6, 40.0), turned to -90 degrees
- moved C301 41.5 mm to (114.8, 53.8)
- moved R202 40.2 mm to (146.8, 35.5)
- moved SW202 39.5 mm to (131.5, 46.0), turned to 90 degrees
- moved R205 39.5 mm to (142.6, 40.0), turned to -90 degrees
- moved R201 39.3 mm to (146.8, 34.5)
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- renumbered C1002 to C101, C1001 to C102, C2001 to C201, C2002 to C202, C2003 to C203, C2004 to C204, C2005 to C205, C2006 to C206, C2007 to C207, C2008 to C208, C2009 to C209, C2010 to C210, C2011 to C211, C2012 to C212, C2013 to C213, C2014 to C214, C2015 to C215, C3011 to C303, C3012 to C304, C3013 to C305, C3014 to C306, C3001 to C307, C3003 to C309, C3004 to C310, C3005 to C311, C3007 to C313, C3008 to C314, D2001 to D201, F3001 to F301, J1002 to J101, J5 to J102, J1001 to J103, J2002 to J201, J2001 to J202, J3001 to J301, J3002 to J302, JP3001 to JP301, L3001 to L301, L3002 to L302, R2001 to R201, R2002 to R202, R2003 to R203, R2004 to R204, R2005 to R205, R2006 to R206, R2007 to R207, R3001 to R301, R3002 to R302, R3003 to R303, R3004 to R304, R3005 to R305, SW2001 to SW201, SW2002 to SW202, TP3003 to TP301, TP3001 to TP302, TP3002 to TP303, U2001 to U201, U2002 to U202, U3003 to U301, U3004 to U302, U3001 to U303, U3002 to U304, Y2001 to Y201, Y3001 to Y301
Connections:
- C305 pad 2: Net-(U3004-OSC2) -> Net-(U302-OSC2)
- U202 pad 27: /Microcontroller/GPIO16 -> /MISO
- U202 pad 28: /Microcontroller/GPIO17 -> /~{CS}
- U202 pad 29: /Microcontroller/GPIO18 -> /SCK
- U202 pad 30: /Microcontroller/GPIO19 -> /MOSI
- U202 pad 32: /Microcontroller/GPIO21 -> /BTN_RIGHT
- U202 pad 34: /Microcontroller/GPIO22 -> /BTN_LEFT
- U202 pad 37: /Microcontroller/GPIO25 -> /BTN
- U202 pad 38: /Microcontroller/GPIO26_ADC0 -> /VR_y
- U202 pad 39: /Microcontroller/GPIO27_ADC1 -> /VR_x
- U202 pad 6: /Microcontroller/GPIO4 -> /SDA
- U202 pad 7: /Microcontroller/GPIO5 -> /SCL
- U302 pad 14: /CAN_Bus+power/SCK -> /SCK
- U302 pad 16: /CAN_Bus+power/MOSI -> /MOSI
- U302 pad 17: /CAN_Bus+power/MISO -> /MISO
- U302 pad 18: /CAN_Bus+power/~{CS} -> /~{CS}
- U302 pad 8: Net-(U3004-OSC2) -> Net-(U302-OSC2)
- Y301 pad 3: GND -> Net-(U302-OSC2)
- Y301 pad 4: Net-(U3004-OSC2) -> GND
Routing:
- net /CAN_Bus+power/CANH: track 0.00 -> 44.3 mm
- net /MOSI: track 0.00 -> 41.7 mm, vias 0 -> 2
- net /~{CS}: track 0.00 -> 39.7 mm, vias 0 -> 2
- net /MISO: track 0.00 -> 38.7 mm, vias 0 -> 2
- net /SCK: track 0.00 -> 38.0 mm, vias 0 -> 2
- net /CAN_Bus+power/CANL: track 0.00 -> 36.5 mm
- net +1V1: track 0.00 -> 28.8 mm, vias 0 -> 3
- net /SDA: track 0.00 -> 28.2 mm, vias 0 -> 1
- net /SCL: track 0.00 -> 24.4 mm, vias 0 -> 1
- net /BTN: track 0.00 -> 21.8 mm
- net /VR_x: track 0.00 -> 20.4 mm
- net /VR_y: track 0.00 -> 20.2 mm
- net /BTN_LEFT: track 0.00 -> 19.0 mm, vias 0 -> 2
- net /BTN_RIGHT: track 0.00 -> 16.3 mm, vias 0 -> 2
- net +5V: track 0.00 -> 16.0 mm, vias 0 -> 10
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- added copper zone on F.Cu, net +3V3
- added copper zone on In2.Cu, net +3V3
- added copper zone on F.Cu, net +5V
- added copper zone on In2.Cu, net +5V
- added copper zone on F.Cu, net +SYSTEM
- added copper zone on B.Cu, net GND
- added copper zone on F.Cu, net GND
- added copper zone on In1.Cu, net GND
- added copper zone on In1.Cu, net Net-(F301-Pad1)
- added copper zone on F.Cu, net Net-(U303-SW)
- added copper zone on F.Cu, net Net-(U304-SW)
Other:
- board outline added: 66.8 x 26 mm
- copper layers 2 -> 4
- board text added: "3V3"
- board text added: "5V"
- board text added: "BOOT"
- board text added: "CAN TERM"
- board text added: "EENX16-VT24-27 User Interface Module"
- board text added: "RESET"

Commit message: Changes and fixes
Parts:
- Y201: footprint Crystal:Crystal_SMD_Abracon_ABM3B-4Pin_5.0x3.2mm -> Crystal:Crystal_SMD_2520-4Pin_2.5x2.0mm
- moved Y201 1.45 mm to (135.7, 52.4)
Routing:
- net GND: vias 113 -> 106

Commit message: final fixes (hopefully) (GONE WRONG?!) (real)
Parts:
- moved R201 0.25 mm to (146.8, 34.2)
- moved R202 0.25 mm to (146.8, 35.2)
Routing:
- net +1V1: track 28.8 -> 29.7 mm
Other:
- board text added: "JLCJLCJLCJLC"

Commit message: Add software files
Parts:
- moved C215 0.05 mm to (130.5, 52.7)
Changed lines of the file:
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@@
 	(footprint "Capacitor_SMD:C_0402_1005Metric"
 		(layer "F.Cu")
-		(at 130.55 52.7 -90)
+		(at 130.5 52.7 -90)
 		(descr "Capacitor SMD 0402 (1005 Metric), square (rectangular) end terminal, IPC_7351 nominal, (Body size source: IPC-SM-782 page 76, https://www.pcb-3d.com/wordpress/wp-content/uploads/ipc-sm-782a_amendment_1_and_2.pdf), generated with kicad-footprint-generator")
 		(tags "capacitor")
